Commit message: [Beetle][Hand] modified urdf to enable hand grasping in simulation

File: robots/beetle/robots/beetle_hand.urdf.xacro (robot description, xacro)
@@ -11,12 +11,12 @@
   ##### dummy grasp links ####
   <joint name="base_dummy_arm_joint" type="fixed">
-    <parent link="base_link"/>
+    <parent link="hand_palm"/>
     <child link="dummy_arm"/>
-    <origin xyz="0.22 0 0.1455" rpy="0 0 0"/>
+    <origin xyz="0.0 0 0.0" rpy="0 0 0"/>
   </joint>
   <link name="dummy_arm">
     <inertial>
       <mass value = "0.01" />
-      <origin xyz="0.05 0 0" rpy="0 0 0"/>
+      <origin xyz="0.00 0 0" rpy="0 0 0"/>
       <inertia
           ixx="0.0001" ixy="0.0000" ixz="0.0000"
@@ -27,5 +27,5 @@
     <parent link="dummy_arm"/>
     <child link="dummy_palm"/>
-    <origin xyz="0.02 0 0" rpy="0 0 0"/>
+    <origin xyz="0.00 0 0" rpy="0 0 0"/>
     <axis xyz="1 0 0"/>
     <limit lower="0" upper="0" effort="0" velocity="0"/>
@@ -147,10 +147,28 @@
       </geometry>
     </visual>
-    <collision>
-      <origin xyz="0.01215 0 0.022" rpy="0 0 0"/>
-      <geometry>
-  	<box size="0.283 0.071 0.118"/>
-      </geometry>
-    </collision>
+    <!-- <collision> -->
+    <!--   <origin xyz="0.01215 0 0.022" rpy="0 0 0"/> -->
+    <!--   <geometry> -->
+    <!-- 	<box size="0.283 0.071 0.118"/> -->
+    <!--   </geometry> -->
+    <!-- </collision> -->
+  </link>
+  <joint name="hand_palm_joint" type="revolute">
+    <child link="hand_palm"/>
+    <parent link="hand"/>
+    <limit lower="0" upper="0" effort="0" velocity="0"/>
+    <dynamics damping="0.2" friction="0.02"/>
+    <origin xyz="0.246 0 0.03" rpy="0 0 0"/>
+    <axis xyz="1 0 0"/>
+  </joint>
+  <link name="hand_palm">
+    <inertial>
+      <origin xyz="0.0 0.0 0.0"/>
+      <mass value="0.00001"/>
+      <inertia
+  	  ixx="0.00001" ixy="0.00000" ixz="0.0000001"
+  	  iyy="0.00001" iyz="0.00000"
+  	  izz="0.00001"/>
+    </inertial>
   </link>
   <link name="hand_2">
@@ -169,10 +187,10 @@
       </geometry>
     </visual>
-    <collision>
-      <origin xyz="0.01215 0 0.022" rpy="0 0 0"/>
-      <geometry>
-  	<box size="0.283 0.071 0.118"/>
-      </geometry>
-    </collision>
+    <!-- <collision> -->
+    <!--   <origin xyz="0.01215 0 0.022" rpy="0 0 0"/> -->
+    <!--   <geometry> -->
+    <!-- 	<box size="0.283 0.071 0.118"/> -->
+    <!--   </geometry> -->
+    <!-- </collision> -->
   </link>
   ## beetle hand joint

Commit message: [Beetle][Hand] modified for processing addExtraModule service

File: robots/beetle/robots/beetle_hand.urdf.xacro (robot description, xacro)
@@ -11,12 +11,12 @@
   ##### dummy grasp links ####
   <joint name="base_dummy_arm_joint" type="fixed">
-    <parent link="hand_palm"/>
+    <parent link="base_link"/>
     <child link="dummy_arm"/>
-    <origin xyz="0.0 0 0.0" rpy="0 0 0"/>
+    <origin xyz="0.22 0 0.1455" rpy="0 0 0"/>
   </joint>
   <link name="dummy_arm">
     <inertial>
       <mass value = "0.01" />
-      <origin xyz="0.00 0 0" rpy="0 0 0"/>
+      <origin xyz="0.05 0 0" rpy="0 0 0"/>
       <inertia
           ixx="0.0001" ixy="0.0000" ixz="0.0000"
@@ -27,5 +27,5 @@
     <parent link="dummy_arm"/>
     <child link="dummy_palm"/>
-    <origin xyz="0.00 0 0" rpy="0 0 0"/>
+    <origin xyz="0.02 0 0" rpy="0 0 0"/>
     <axis xyz="1 0 0"/>
     <limit lower="0" upper="0" effort="0" velocity="0"/>
@@ -50,4 +50,5 @@
     <parent link="dummy_palm"/>
     <child link="dummy_gripper"/>
+    <!-- <child link="plusx_dummy_gripper"/> -->
     <origin xyz="0 0 0" rpy="0 0 0"/>
     <axis xyz="1 0 0"/>
@@ -56,4 +57,5 @@
   </joint>
   <link name="dummy_gripper">
+  <!-- <link name="plusx_dummy_gripper"> -->
     <inertial>
       <mass value = "0.001" />
@@ -147,28 +149,10 @@
       </geometry>
     </visual>
-    <!-- <collision> -->
-    <!--   <origin xyz="0.01215 0 0.022" rpy="0 0 0"/> -->
-    <!--   <geometry> -->
-    <!-- 	<box size="0.283 0.071 0.118"/> -->
-    <!--   </geometry> -->
-    <!-- </collision> -->
-  </link>
-  <joint name="hand_palm_joint" type="revolute">
-    <child link="hand_palm"/>
-    <parent link="hand"/>
-    <limit lower="0" upper="0" effort="0" velocity="0"/>
-    <dynamics damping="0.2" friction="0.02"/>
-    <origin xyz="0.246 0 0.03" rpy="0 0 0"/>
-    <axis xyz="1 0 0"/>
-  </joint>
-  <link name="hand_palm">
-    <inertial>
-      <origin xyz="0.0 0.0 0.0"/>
-      <mass value="0.00001"/>
-      <inertia
-  	  ixx="0.00001" ixy="0.00000" ixz="0.0000001"
-  	  iyy="0.00001" iyz="0.00000"
-  	  izz="0.00001"/>
-    </inertial>
+    <collision>
+      <origin xyz="0.01215 0 0.022" rpy="0 0 0"/>
+      <geometry>
+  	<box size="0.283 0.071 0.118"/>
+      </geometry>
+    </collision>
   </link>
   <link name="hand_2">
@@ -187,10 +171,10 @@
       </geometry>
     </visual>
-    <!-- <collision> -->
-    <!--   <origin xyz="0.01215 0 0.022" rpy="0 0 0"/> -->
-    <!--   <geometry> -->
-    <!-- 	<box size="0.283 0.071 0.118"/> -->
-    <!--   </geometry> -->
-    <!-- </collision> -->
+    <collision>
+      <origin xyz="0.01215 0 0.022" rpy="0 0 0"/>
+      <geometry>
+  	<box size="0.283 0.071 0.118"/>
+      </geometry>
+    </collision>
   </link>
   ## beetle hand joint

Commit message: [Beetle][Hand] Modified for fix the hand position

File: robots/beetle/robots/beetle_hand.urdf.xacro (robot description, xacro)
@@ -14,5 +14,6 @@
     <parent link="base_link"/>
     <child link="dummy_arm_1"/>
-    <origin xyz="0.22 0 0.1455" rpy="0 0 0"/>
+    <!-- <origin xyz="0.22 0 0.1455" rpy="0 0 0"/> -->
+    <origin xyz="0.272 0 0.153" rpy="0 0 0"/>
   </joint>
   <link name="dummy_arm_1">
@@ -83,5 +84,6 @@
     <parent link="base_link"/>
     <child link="dummy_arm_2"/>
-    <origin xyz="-0.22 0 0.1455" rpy="0 0 ${pi}"/>
+    <!-- <origin xyz="-0.22 0 0.1455" rpy="0 0 ${pi}"/> -->
+    <origin xyz="-0.272 0 0.153" rpy="0 0 ${pi}"/>
   </joint>
   <link name="dummy_arm_2">
@@ -209,12 +211,16 @@
       <mass value="0.3900000"/>
       <inertia
-  	  ixx="0.000699" ixy="-0.000004" ixz="0.000769"
-  	  iyy="0.005953" iyz="-0.000005"
-  	  izz="0.00541"/>
-    </inertial>
-    <visual>
-      <origin xyz="0 0 0" rpy="0 0 0"/>
-      <geometry>
-    	<mesh filename="package://beetle/urdf/mesh/beetle_hand_handmech_all.dae"/>
+  	  ixx="0.000911" ixy="0.001204" ixz="0.000002"
+  	  iyy="0.009690" iyz="-0.000005"
+  	  izz="0.010438"/>
+      <!-- <inertia -->
+      <!-- 	  ixx="0.000699" ixy="-0.000004" ixz="0.000769" -->
+      <!-- 	  iyy="0.005953" iyz="-0.000005" -->
+      <!-- 	  izz="0.00541"/> -->
+    </inertial>
+    <visual>
+      <origin xyz="0 0 0" rpy="0 0 0"/>
+      <geometry>
+    	<mesh filename="package://beetle/urdf/mesh/hand9_handmech_all.dae" scale="0.1 0.1 0.1"/>
       </geometry>
     </visual>
@@ -231,12 +237,16 @@
       <mass value="0.3900000"/>
       <inertia
-  	  ixx="0.000699" ixy="-0.000004" ixz="0.000769"
-  	  iyy="0.005953" iyz="-0.000005"
-  	  izz="0.00541"/>
-    </inertial>
-    <visual>
-      <origin xyz="0 0 0" rpy="0 0 0"/>
-      <geometry>
-    	<mesh filename="package://beetle/urdf/mesh/beetle_hand_handmech_all.dae"/>
+  	  ixx="0.000911" ixy="0.001204" ixz="0.000002"
+  	  iyy="0.009690" iyz="-0.000005"
+  	  izz="0.010438"/>
+      <!-- <inertia -->
+      <!-- 	  ixx="0.000699" ixy="-0.000004" ixz="0.000769" -->
+      <!-- 	  iyy="0.005953" iyz="-0.000005" -->
+      <!-- 	  izz="0.00541"/> -->
+    </inertial>
+    <visual>
+      <origin xyz="0 0 0" rpy="0 0 0"/>
+      <geometry>
+    	<mesh filename="package://beetle/urdf/mesh/hand9_handmech_all.dae" scale="0.1 0.1 0.1"/>
       </geometry>
     </visual>

Commit message: [Beetle][Hand] Modified for using in real robot

File: robots/beetle/robots/beetle_hand.urdf.xacro (robot description, xacro)
@@ -29,5 +29,5 @@
     <parent link="dummy_arm_1"/>
     <child link="dummy_palm_1"/>
-    <origin xyz="0.02 0 0" rpy="0 0 0"/>
+    <origin xyz="0 0 0" rpy="0 0 0"/>
     <axis xyz="1 0 0"/>
     <limit lower="0" upper="0" effort="0" velocity="0"/>
@@ -99,5 +99,5 @@
     <parent link="dummy_arm_2"/>
     <child link="dummy_palm_2"/>
-    <origin xyz="0.02 0 0" rpy="0 0 0"/>
+    <origin xyz="0 0 0" rpy="0 0 0"/>
     <axis xyz="1 0 0"/>
     <limit lower="0" upper="0" effort="0" velocity="0"/>
