Commit message: [Beatle]{Hand] modified for dual and model

File: robots/beetle/robots/beetle_hand.gazebo.xacro (robot description, xacro)
@@ -9,9 +9,17 @@
   <!-- gazebo plugin for docking mech -->
   <gazebo>
-    <plugin name="gazebo_grasp_fix" filename="libgazebo_grasp_fix.so">
+    <plugin name="gazebo_grasp_fix_1" filename="libgazebo_grasp_fix.so">
       <arm>
-        <arm_name>docking_mech</arm_name>
-        <palm_link>dummy_palm</palm_link>
-        <gripper_link>dummy_gripper</gripper_link>
+        <arm_name>docking_mech_1</arm_name>
+        <palm_link>dummy_palm_1</palm_link>
+        <gripper_link>dummy_gripper_1</gripper_link>
+	<arm_name>docking_mech_2</arm_name>
+        <palm_link>dummy_palm_2</palm_link>
+        <gripper_link>dummy_gripper_2</gripper_link>
+      </arm>
+      <arm>
+	<arm_name>docking_mech_2</arm_name>
+        <palm_link>dummy_palm_2</palm_link>
+        <gripper_link>dummy_gripper_2</gripper_link>
       </arm>
       <forces_angle_tolerance>90</forces_angle_tolerance>

File: robots/beetle/robots/beetle_hand.urdf.xacro (robot description, xacro)
@@ -10,10 +10,11 @@
   <xacro:beetle_thrust_link self="4" rotor_direction="1"/>
   ##### dummy grasp links ####
-  <joint name="base_dummy_arm_joint" type="fixed">
-    <parent link="base_link"/>
-    <child link="dummy_arm"/>
+  <!-- dummy_hand 1-->
+  <joint name="base_dummy_arm_1_joint" type="fixed">
+    <parent link="base_link"/>
+    <child link="dummy_arm_1"/>
     <origin xyz="0.22 0 0.1455" rpy="0 0 0"/>
   </joint>
-  <link name="dummy_arm">
+  <link name="dummy_arm_1">
     <inertial>
       <mass value = "0.01" />
@@ -24,7 +25,7 @@
     </inertial>
   </link>
-  <joint name="dummy_arm_palm_joint" type="revolute">
-    <parent link="dummy_arm"/>
-    <child link="dummy_palm"/>
+  <joint name="dummy_arm_1_palm_joint" type="revolute">
+    <parent link="dummy_arm_1"/>
+    <child link="dummy_palm_1"/>
     <origin xyz="0.02 0 0" rpy="0 0 0"/>
     <axis xyz="1 0 0"/>
@@ -32,23 +33,23 @@
     <dynamics damping="0.2" friction="0.02"/>
   </joint>
-  <link name="dummy_palm">
-    <inertial>
-      <mass value = "0.001" />
-      <origin xyz="0 0 0" rpy="0 0 0"/>
-      <inertia
-          ixx="0.0001" ixy="0.0000" ixz="0.0000"
-          iyy="0.0001" iyz="0.0000" izz="0.0001"/>
-    </inertial>
-    <collision>
-      <origin xyz="0 0 0" rpy="0 0 0"/>
-      <geometry>
-        <box size="0.01 0.01 0.01"/>
-      </geometry>
-    </collision>
-  </link>
-  <joint name="dummy_palm_gripper_joint" type="revolute">
-    <parent link="dummy_palm"/>
-    <child link="dummy_gripper"/>
-    <!-- <child link="plusx_dummy_gripper"/> -->
+  <link name="dummy_palm_1">
+    <inertial>
+      <mass value = "0.001" />
+      <origin xyz="0 0 0" rpy="0 0 0"/>
+      <inertia
+          ixx="0.0001" ixy="0.0000" ixz="0.0000"
+          iyy="0.0001" iyz="0.0000" izz="0.0001"/>
+    </inertial>
+    <collision>
+      <origin xyz="0 0 0" rpy="0 0 0"/>
+      <geometry>
+        <box size="0.01 0.01 0.01"/>
+      </geometry>
+    </collision>
+  </link>
+  <joint name="dummy_palm_gripper_joint_1" type="revolute">
+    <parent link="dummy_palm_1"/>
+    <child link="dummy_gripper_1"/>
+    <!-- <child link="plusx_dummy_gripper_1"/> -->
     <origin xyz="0 0 0" rpy="0 0 0"/>
     <axis xyz="1 0 0"/>
@@ -56,6 +57,75 @@
     <dynamics damping="0.2" friction="0.02"/>
   </joint>
-  <link name="dummy_gripper">
-  <!-- <link name="plusx_dummy_gripper"> -->
+  <link name="dummy_gripper_1">
+  <!-- <link name="plusx_dummy_gripper_1"> -->
+    <inertial>
+      <mass value = "0.001" />
+      <origin xyz="0 0 0" rpy="0 0 0"/>
+      <inertia
+          ixx="0.0001" ixy="0.0000" ixz="0.0000"
+          iyy="0.0001" iyz="0.0000" izz="0.0001"/>
+    </inertial>
+    <collision>
+      <origin xyz="0 0 0" rpy="0 0 0"/>
+      <geometry>
+        <box size="0.01 0.01 0.01"/>
+      </geometry>
+    </collision>
+    <visual>
+      <origin xyz="0 0 0" rpy="0.0 0 0"/>
+      <geometry>
+        <box size="0.01 0.01 0.01"/>
+      </geometry>
+    </visual>
+  </link>
+  <!-- dummy_hand 2-->
+  <joint name="base_dummy_arm_2_joint" type="fixed">
+    <parent link="base_link"/>
+    <child link="dummy_arm_2"/>
+    <origin xyz="-0.22 0 0.1455" rpy="0 0 ${pi}"/>
+  </joint>
+  <link name="dummy_arm_2">
+    <inertial>
+      <mass value = "0.01" />
+      <origin xyz="0.05 0 0" rpy="0 0 0"/>
+      <inertia
+          ixx="0.0001" ixy="0.0000" ixz="0.0000"
+          iyy="0.0001" iyz="0.0000" izz="0.0001"/>
+    </inertial>
+  </link>
+  <joint name="dummy_arm_2_palm_joint" type="revolute">
+    <parent link="dummy_arm_2"/>
+    <child link="dummy_palm_2"/>
+    <origin xyz="0.02 0 0" rpy="0 0 0"/>
+    <axis xyz="1 0 0"/>
+    <limit lower="0" upper="0" effort="0" velocity="0"/>
+    <dynamics damping="0.2" friction="0.02"/>
+  </joint>
+  <link name="dummy_palm_2">
+    <inertial>
+      <mass value = "0.001" />
+      <origin xyz="0 0 0" rpy="0 0 0"/>
+      <inertia
+          ixx="0.0001" ixy="0.0000" ixz="0.0000"
+          iyy="0.0001" iyz="0.0000" izz="0.0001"/>
+    </inertial>
+    <collision>
+      <origin xyz="0 0 0" rpy="0 0 0"/>
+      <geometry>
+        <box size="0.01 0.01 0.01"/>
+      </geometry>
+    </collision>
+  </link>
+  <joint name="dummy_palm_gripper_joint_2" type="revolute">
+    <parent link="dummy_palm_2"/>
+    <child link="dummy_gripper_2"/>
+    <!-- <child link="plusx_dummy_gripper_2"/> -->
+    <origin xyz="0 0 0" rpy="0 0 0"/>
+    <axis xyz="1 0 0"/>
+    <limit lower="0" upper="0" effort="0" velocity="0"/>
+    <dynamics damping="0.2" friction="0.02"/>
+  </joint>
+  <link name="dummy_gripper_2">
+    <!-- <link name="plusx_dummy_gripper_2"> -->
     <inertial>
       <mass value = "0.001" />

Commit message: [Beetle][Hand] Modified for simulate camera in gazebo

File: robots/beetle/robots/beetle_hand.gazebo.xacro (robot description, xacro)
@@ -32,3 +32,68 @@
     </plugin>
   </gazebo>
+  <gazebo reference="base_link">
+    <mu1>0.1</mu1>
+    <mu2>0.1</mu2>
+  </gazebo>
+  <!-- <!-\- sensors -\-> -->
+  <!-- <xacro:extra_module name = "downward_camera_frame" parent = "base_link"> -->
+  <!--   <origin xyz="0.270 0.002 0.078" rpy="0 0 0"/> -->
+  <!--   <inertial> -->
+  <!--     <mass value = "0.00001" /> -->
+  <!--     <origin xyz="0 0 0" rpy="0 0 0"/> -->
+  <!--     <inertia -->
+  <!--         ixx="0.000001" ixy="0.0" ixz="0.0" -->
+  <!--         iyy="0.000001" iyz="0.0" -->
+  <!--         izz="0.000002"/> -->
+  <!--   </inertial> -->
+  <!-- </xacro:extra_module> -->
+  <!-- <xacro:extra_module name = "downward_camera_optical_frame" parent = "downward_camera_frame"> -->
+  <!--   <origin xyz="0 0 0" rpy="${-pi / 2} 0 ${-pi / 2}"/> -->
+  <!--   <inertial> -->
+  <!--     <mass value = "0.00001" /> -->
+  <!--     <origin xyz="0 0 0" rpy="0 0 0"/> -->
+  <!--     <inertia -->
+  <!--         ixx="0.000001" ixy="0.0" ixz="0.0" -->
+  <!--         iyy="0.000001" iyz="0.0" -->
+  <!--         izz="0.000002"/> -->
+  <!--   </inertial> -->
+  <!-- </xacro:extra_module> -->
+  <!-- <!-\- gazebo plugin for camera module -\->   -->
+  <!-- <gazebo reference="downward_camera_frame"> -->
+  <!--   <sensor type="camera" name="downward_camera"> -->
+  <!--     <update_rate>30.0</update_rate> -->
+  <!--     <camera name="head"> -->
+  <!--       <horizontal_fov>1.57</horizontal_fov> -->
+  <!--       <image> -->
+  <!--         <width>640</width> -->
+  <!--         <height>480</height> -->
+  <!--         <format>R8G8B8</format> -->
+  <!--       </image> -->
+  <!--       <clip> -->
+  <!--         <near>0.02</near> -->
+  <!--         <far>300</far> -->
+  <!--       </clip> -->
+  <!--       <noise> -->
+  <!--         <type>gaussian</type> -->
+  <!--         <mean>0.0</mean> -->
+  <!--         <stddev>0.007</stddev> -->
+  <!--       </noise> -->
+  <!--     </camera> -->
+  <!--     <plugin name="camera_controller" filename="libgazebo_ros_camera.so"> -->
+  <!--       <robotNamespace>$(arg robot_name)</robotNamespace> -->
+  <!--       <alwaysOn>true</alwaysOn> -->
+  <!--       <updateRate>0.0</updateRate> -->
+  <!--       <cameraName>downward_camera</cameraName> -->
+  <!--       <imageTopicName>image_raw</imageTopicName> -->
+  <!--       <cameraInfoTopicName>camera_info</cameraInfoTopicName> -->
+  <!--       <frameName>downward_camera_optical_frame</frameName> -->
+  <!--       <hackBaseline>0.07</hackBaseline> -->
+  <!--       <distortionK1>0.0</distortionK1> -->
+  <!--       <distortionK2>0.0</distortionK2> -->
+  <!--       <distortionK3>0.0</distortionK3> -->
+  <!--       <distortionT1>0.0</distortionT1> -->
+  <!--       <distortionT2>0.0</distortionT2> -->
+  <!--     </plugin> -->
+  <!--   </sensor> -->
+  <!-- </gazebo> -->
 </robot>

File: robots/beetle/urdf/common.xacro (robot description, xacro)
@@ -20,3 +20,21 @@
     </gazebo>
   </xacro:macro>
+  <!-- <!-\- extra_module -\-> -->
+  <!-- <xacro:macro name="extra_module" params="name parent *origin *inertial visible:=0 model_url:=0"> -->
+  <!--   <joint name="${parent}2${name}" type="fixed"> -->
+  <!--     <parent link="${parent}"/> -->
+  <!--     <child link="${name}"/> -->
+  <!--     <xacro:insert_block name="origin" /> -->
+  <!--   </joint> -->
+  <!--   <link name="${name}"> -->
+  <!--     <xacro:insert_block name="inertial" /> -->
+  <!--     <xacro:if value="${visible == 1}"> -->
+  <!--       <visual> -->
+  <!--         <geometry> -->
+  <!--           <mesh filename="${model_url}"/> -->
+  <!--         </geometry> -->
+  <!--       </visual> -->
+  <!--     </xacro:if> -->
+  <!--   </link> -->
+  <!-- </xacro:macro> -->
 </robot>

Commit message: [Beetle][Hand] modified for doubletag_detection flightnav and add camera on gazebo

File: robots/beetle/robots/beetle_hand.gazebo.xacro (robot description, xacro)
@@ -36,64 +36,70 @@
     <mu2>0.1</mu2>
   </gazebo>
-  <!-- <!-\- sensors -\-> -->
-  <!-- <xacro:extra_module name = "downward_camera_frame" parent = "base_link"> -->
-  <!--   <origin xyz="0.270 0.002 0.078" rpy="0 0 0"/> -->
-  <!--   <inertial> -->
-  <!--     <mass value = "0.00001" /> -->
-  <!--     <origin xyz="0 0 0" rpy="0 0 0"/> -->
-  <!--     <inertia -->
-  <!--         ixx="0.000001" ixy="0.0" ixz="0.0" -->
-  <!--         iyy="0.000001" iyz="0.0" -->
-  <!--         izz="0.000002"/> -->
-  <!--   </inertial> -->
-  <!-- </xacro:extra_module> -->
-  <!-- <xacro:extra_module name = "downward_camera_optical_frame" parent = "downward_camera_frame"> -->
-  <!--   <origin xyz="0 0 0" rpy="${-pi / 2} 0 ${-pi / 2}"/> -->
-  <!--   <inertial> -->
-  <!--     <mass value = "0.00001" /> -->
-  <!--     <origin xyz="0 0 0" rpy="0 0 0"/> -->
-  <!--     <inertia -->
-  <!--         ixx="0.000001" ixy="0.0" ixz="0.0" -->
-  <!--         iyy="0.000001" iyz="0.0" -->
-  <!--         izz="0.000002"/> -->
-  <!--   </inertial> -->
-  <!-- </xacro:extra_module> -->
-  <!-- <!-\- gazebo plugin for camera module -\->   -->
-  <!-- <gazebo reference="downward_camera_frame"> -->
-  <!--   <sensor type="camera" name="downward_camera"> -->
-  <!--     <update_rate>30.0</update_rate> -->
-  <!--     <camera name="head"> -->
-  <!--       <horizontal_fov>1.57</horizontal_fov> -->
-  <!--       <image> -->
-  <!--         <width>640</width> -->
-  <!--         <height>480</height> -->
-  <!--         <format>R8G8B8</format> -->
-  <!--       </image> -->
-  <!--       <clip> -->
-  <!--         <near>0.02</near> -->
-  <!--         <far>300</far> -->
-  <!--       </clip> -->
-  <!--       <noise> -->
-  <!--         <type>gaussian</type> -->
-  <!--         <mean>0.0</mean> -->
-  <!--         <stddev>0.007</stddev> -->
-  <!--       </noise> -->
-  <!--     </camera> -->
-  <!--     <plugin name="camera_controller" filename="libgazebo_ros_camera.so"> -->
-  <!--       <robotNamespace>$(arg robot_name)</robotNamespace> -->
-  <!--       <alwaysOn>true</alwaysOn> -->
-  <!--       <updateRate>0.0</updateRate> -->
-  <!--       <cameraName>downward_camera</cameraName> -->
-  <!--       <imageTopicName>image_raw</imageTopicName> -->
-  <!--       <cameraInfoTopicName>camera_info</cameraInfoTopicName> -->
-  <!--       <frameName>downward_camera_optical_frame</frameName> -->
-  <!--       <hackBaseline>0.07</hackBaseline> -->
-  <!--       <distortionK1>0.0</distortionK1> -->
-  <!--       <distortionK2>0.0</distortionK2> -->
-  <!--       <distortionK3>0.0</distortionK3> -->
-  <!--       <distortionT1>0.0</distortionT1> -->
-  <!--       <distortionT2>0.0</distortionT2> -->
-  <!--     </plugin> -->
-  <!--   </sensor> -->
-  <!-- </gazebo> -->
+  <gazebo reference="apriltag_0">
+    <material>Apriltag36_11_00000</material>
+  </gazebo>
+  <gazebo reference="apriltag_1">
+    <material>Apriltag36_11_00001</material>
+  </gazebo>
+  <!-- sensors -->
+  <xacro:extra_module name = "downward_camera_frame" parent = "base_link">
+    <origin xyz="0.270 0.002 0.078" rpy="0 0 0"/>
+    <inertial>
+      <mass value = "0.00001" />
+      <origin xyz="0 0 0" rpy="0 0 0"/>
+      <inertia
+          ixx="0.000001" ixy="0.0" ixz="0.0"
+          iyy="0.000001" iyz="0.0"
+          izz="0.000002"/>
+    </inertial>
+  </xacro:extra_module>
+  <xacro:extra_module name = "downward_camera_optical_frame" parent = "downward_camera_frame">
+    <origin xyz="0 0 0" rpy="${-pi / 2} 0 ${-pi / 2}"/>
+    <inertial>
+      <mass value = "0.00001" />
+      <origin xyz="0 0 0" rpy="0 0 0"/>
+      <inertia
+          ixx="0.000001" ixy="0.0" ixz="0.0"
+          iyy="0.000001" iyz="0.0"
+          izz="0.000002"/>
+    </inertial>
+  </xacro:extra_module>
+  <!-- gazebo plugin for camera module -->
+  <gazebo reference="downward_camera_frame">
+    <sensor type="camera" name="downward_camera">
+      <update_rate>30.0</update_rate>
+      <camera name="head">
+        <horizontal_fov>1.57</horizontal_fov>
+        <image>
+          <width>640</width>
+          <height>480</height>
+          <format>R8G8B8</format>
+        </image>
+        <clip>
+          <near>0.02</near>
+          <far>300</far>
+        </clip>
+        <noise>
+          <type>gaussian</type>
+          <mean>0.0</mean>
+          <stddev>0.007</stddev>
+        </noise>
+      </camera>
+      <plugin name="camera_controller" filename="libgazebo_ros_camera.so">
+        <robotNamespace>$(arg robot_name)</robotNamespace>
+        <alwaysOn>true</alwaysOn>
+        <updateRate>0.0</updateRate>
+        <cameraName>downward_camera</cameraName>
+        <imageTopicName>image_raw</imageTopicName>
+        <cameraInfoTopicName>camera_info</cameraInfoTopicName>
+        <frameName>downward_camera_optical_frame</frameName>
+        <hackBaseline>0.07</hackBaseline>
+        <distortionK1>0.0</distortionK1>
+        <distortionK2>0.0</distortionK2>
+        <distortionK3>0.0</distortionK3>
+        <distortionT1>0.0</distortionT1>
+        <distortionT2>0.0</distortionT2>
+      </plugin>
+    </sensor>
+  </gazebo>
 </robot>

File: robots/beetle/urdf/beetle_hand.urdf.xacro (robot description, xacro)
@@ -204,3 +204,22 @@
     </transmission>
   </xacro:macro>
+  <!-- extra_module -->
+  <xacro:macro name="extra_module" params="name parent *origin *inertial visible:=0 model_url:=0">
+    <joint name="${parent}2${name}" type="fixed">
+      <parent link="${parent}"/>
+      <child link="${name}"/>
+      <xacro:insert_block name="origin" />
+    </joint>
+    <link name="${name}">
+      <xacro:insert_block name="inertial" />
+      <xacro:if value="${visible == 1}">
+        <visual>
+	  <origin rpy="0 0 0" xyz="0 0 0"/>
+          <geometry>
+            <mesh filename="${model_url}" scale="${scale} ${scale} ${scale}"/>
+          </geometry>
+        </visual>
+      </xacro:if>
+    </link>
+  </xacro:macro>
 </robot>

File: robots/beetle/urdf/common.xacro (robot description, xacro)
@@ -20,21 +20,3 @@
     </gazebo>
   </xacro:macro>
-  <!-- <!-\- extra_module -\-> -->
-  <!-- <xacro:macro name="extra_module" params="name parent *origin *inertial visible:=0 model_url:=0"> -->
-  <!--   <joint name="${parent}2${name}" type="fixed"> -->
-  <!--     <parent link="${parent}"/> -->
-  <!--     <child link="${name}"/> -->
-  <!--     <xacro:insert_block name="origin" /> -->
-  <!--   </joint> -->
-  <!--   <link name="${name}"> -->
-  <!--     <xacro:insert_block name="inertial" /> -->
-  <!--     <xacro:if value="${visible == 1}"> -->
-  <!--       <visual> -->
-  <!--         <geometry> -->
-  <!--           <mesh filename="${model_url}"/> -->
-  <!--         </geometry> -->
-  <!--       </visual> -->
-  <!--     </xacro:if> -->
-  <!--   </link> -->
-  <!-- </xacro:macro> -->
 </robot>
