Commit message: hydrus4rod_in_hole

File: robots/hydrus/urdf/common.xacro (robot description, xacro)
@@ -131,5 +131,5 @@
       <origin rpy="0 0 0" xyz="${link_length} 0 0"/>
   </joint>
-  <link name="end_effector">
+  <!-- <link name="end_effector">
     <inertial>
       <origin xyz="0 0 0" rpy="0 0 0"/>
@@ -152,6 +152,5 @@
         </geometry>
       </visual>
-  </link>
-<!--
+  </link>  -->
   <link name="end_effector">
     <inertial>
@@ -164,16 +163,16 @@
     </inertial>
       <collision>
-        <origin rpy="0 1.57 0" xyz="0.3 0 0"/>
-        <geometry>
-          <cylinder length="0.6" radius="0.01"/>
+        <origin rpy="0 1.57 0" xyz="0.1 0 0"/>
+        <geometry>
+          <cylinder length="0.2" radius="0.01"/>
         </geometry>
       </collision>
       <visual>
-        <origin rpy="0 1.57 0" xyz="0.3 0 0"/>
-        <geometry>
-          <cylinder length="0.6" radius="0.01"/>
+        <origin rpy="0 1.57 0" xyz="0.1 0 0"/>
+        <geometry>
+          <cylinder length="0.2" radius="0.01"/>
         </geometry>
       </visual>
-  </link> -->
+  </link>
   <gazebo reference="end_effector">
     <sensor name="contacts" type="contact">

File: robots/hydrus_xi/urdf/common.xacro (robot description, xacro)
@@ -76,13 +76,13 @@
     </inertial>
       <collision>
-        <origin rpy="0 1.57 0" xyz="0.3 0 0"/>
+        <origin rpy="0 1.57 0" xyz="0.1 0 0"/>
         <geometry>
-          <cylinder length="0.6" radius="0.01"/>
+          <cylinder length="0.2" radius="0.01"/>
         </geometry>
       </collision>
       <visual>
-        <origin rpy="0 1.57 0" xyz="0.3 0 0"/>
+        <origin rpy="0 1.57 0" xyz="0.1 0 0"/>
         <geometry>
-          <cylinder length="0.6" radius="0.01"/>
+          <cylinder length="0.2" radius="0.01"/>
         </geometry>
       </visual>
