Commit message: planning_insert demo for going through a 25mm hole automatically

File: robots/hydrus_xi/urdf/common.xacro (robot description, xacro)
@@ -88,4 +88,23 @@
       </visual>
   </link>
+  <joint name="end_eff" type="fixed">
+      <parent link="end_effector"/>
+      <child link="end_frame"/>
+      <origin rpy="0 0 0" xyz="0.2 0 0"/>
+  </joint>
+  <link name="end_frame">
+      <collision>
+        <origin rpy="0 0 0" xyz="0 0 0"/>
+        <geometry>
+          <sphere radius="0.01"/>
+        </geometry>
+      </collision>
+      <visual>
+        <origin rpy="0 1.57 0" xyz="0 0 0"/>
+        <geometry>
+          <sphere radius="0.01"/>
+        </geometry>
+      </visual>
+  </link>
   <gazebo reference="end_effector">
     <sensor name="contacts" type="contact">

File: robots/hydrus_xi/urdf/wall.urdf (robot description, URDF)
Before this commit: robot aaaa, 1 links, 0 joints
Links:
- added link world
- link wall_link: geometry collision mesh filename=package://hydrus_xi/urdf/mesh/scene/wall_link_25mm.dae; visual mesh filename=package://hydrus_xi/urdf/mesh/scene/wall_link_25mm.dae
Joints:
- added joint joint: type fixed, parent world, child wall_link, origin xyz=2.5 0 1 rpy=0 0 0, axis 0 0 1

Commit message: save

File: robots/hydrus_xi/urdf/common.xacro (robot description, xacro)
@@ -81,4 +81,10 @@
         </geometry>
       </collision>
+      <collision>
+        <origin rpy="0 0 0" xyz="0.2 0 0"/>
+        <geometry>
+          <sphere radius="0.01"/>
+        </geometry>
+      </collision>
       <visual>
         <origin rpy="0 1.57 0" xyz="0.1 0 0"/>
@@ -87,6 +93,12 @@
         </geometry>
       </visual>
+      <visual>
+        <origin rpy="0 0 0" xyz="0.2 0 0"/>
+        <geometry>
+          <sphere radius="0.01"/>
+        </geometry>
+      </visual>
   </link>
-  <joint name="end_eff" type="fixed">
+  <!-- <joint name="end_eff" type="fixed">
       <parent link="end_effector"/>
       <child link="end_frame"/>
@@ -106,9 +118,9 @@
         </geometry>
       </visual>
-  </link>
+  </link> -->
   <gazebo reference="end_effector">
     <sensor name="contacts" type="contact">
         <contact>
-          <collision>link4_fixed_joint_lump__end_effector_collision_1</collision>
+          <collision>link4_fixed_joint_lump__end_effector_collision_2</collision>
         </contact>
         <plugin name="gazebo_ros_bumper_controller" filename="libgazebo_ros_bumper.so">

Commit message: update

File: robots/hydrus_xi/urdf/common.xacro (robot description, xacro)
@@ -31,4 +31,5 @@
     </visual>
   </xacro:macro>
+  <mesh filename="T-motor-CF-14inch-CCW.stl"/>
   <xacro:macro name="link_collision_model">
     <collision>

Commit message: commit for merge

File: robots/hydrus_xi/urdf/common.xacro (robot description, xacro)
@@ -70,5 +70,5 @@
     <inertial>
       <origin xyz="0 0 0" rpy="0 0 1.57"/>
-      <mass value="0.001"/>
+      <mass value="0.050"/>
       <inertia
           ixx="0.0001" ixy="0.0" ixz="0.0"

Commit message: adjust params and test deformation caused by ex force

File: robots/hydrus_xi/urdf/common.xacro (robot description, xacro)
@@ -70,5 +70,5 @@
     <inertial>
       <origin xyz="0 0 0" rpy="0 0 1.57"/>
-      <mass value="0.050"/>
+      <mass value="0.001"/>
       <inertia
           ixx="0.0001" ixy="0.0" ixz="0.0"

Commit message: commit for merge

File: robots/hydrus_xi/urdf/common.xacro (robot description, xacro)
@@ -101,5 +101,5 @@
       </visual>
   </link>
-  <!-- <joint name="end_eff" type="fixed">
+  <joint name="end_eff" type="fixed">
       <parent link="end_effector"/>
       <child link="end_frame"/>
@@ -113,11 +113,5 @@
         </geometry>
       </collision>
-      <visual>
-        <origin rpy="0 1.57 0" xyz="0 0 0"/>
-        <geometry>
-          <sphere radius="0.01"/>
-        </geometry>
-      </visual>
-  </link> -->
+  </link>
   <gazebo reference="end_effector">
     <sensor name="contacts" type="contact">

Commit message: Maybe fixed the static error problem by adjusting model

File: robots/hydrus_xi/urdf/common.xacro (robot description, xacro)
@@ -14,6 +14,6 @@
   <xacro:property name="rotor_radius" value=".0178"/>
   <!-- mass [Kg] -->
-  <xacro:property name="rotor_mass" value="0.02"/> <!-- exclude from center mass -->
-  <xacro:property name="bat_mass" value="0.193"/> <!-- 1300mAh -->
+  <xacro:property name="rotor_mass" value="0.13"/> <!-- exclude from center mass -->
+  <xacro:property name="bat_mass" value="0.2"/> <!-- 1300mAh -->
   <!-- dynamics -->
   <m_f_rate value="-0.0182" /> <!-- MN4010KV475_Afro_15inch -->
@@ -72,7 +72,7 @@
       <mass value="0.001"/>
       <inertia
-          ixx="0.0001" ixy="0.0" ixz="0.0"
-          iyy="0.0001" iyz="0.0"
-          izz="0.0001"/>
+          ixx="1e-6" ixy="0.0" ixz="0.0"
+          iyy="1e-6" iyz="0.0"
+          izz="1e-6"/>
     </inertial>
       <collision>

Commit message: redo motor_test and briefly modified data, now the static error problem can be ignored

File: robots/hydrus_xi/urdf/common.xacro (robot description, xacro)
@@ -14,6 +14,6 @@
   <xacro:property name="rotor_radius" value=".0178"/>
   <!-- mass [Kg] -->
-  <xacro:property name="rotor_mass" value="0.13"/> <!-- exclude from center mass -->
-  <xacro:property name="bat_mass" value="0.2"/> <!-- 1300mAh -->
+  <xacro:property name="rotor_mass" value="0.02"/> <!-- exclude from center mass -->
+  <xacro:property name="bat_mass" value="0.05"/> <!-- 1300mAh -->
   <!-- dynamics -->
   <m_f_rate value="-0.0182" /> <!-- MN4010KV475_Afro_15inch -->
@@ -70,5 +70,5 @@
     <inertial>
       <origin xyz="0 0 0" rpy="0 0 1.57"/>
-      <mass value="0.001"/>
+      <mass value="0.07"/>
       <inertia
           ixx="1e-6" ixy="0.0" ixz="0.0"

Commit message: Compelete impedance experiment, save parameters

File: robots/hydrus_xi/urdf/common.xacro (robot description, xacro)
@@ -69,6 +69,6 @@
   <link name="end_effector">
     <inertial>
-      <origin xyz="0 0 0" rpy="0 0 1.57"/>
-      <mass value="0.07"/>
+      <origin xyz="0.00 0 0" rpy="0 0 1.57"/>
+      <mass value="0.02"/>
       <inertia
           ixx="1e-6" ixy="0.0" ixz="0.0"
