Commit message: [Spinal][PWM] Modified condition to judge external pwm device

File: robots/gimbalrotor/urdf/beetle/gimbalrotor.urdf.xacro (robot description, xacro)
@@ -24,14 +24,14 @@
       <inertial>
         <origin xyz="0.000169 0.002346 0.106123" rpy="0 0 0"/>
-        <mass value="1.37825"/>
-        <inertia
-            ixx="0.046756" ixy="0.000586" ixz="0.000055"
-	    iyy="0.063216" iyz="0.000219"
-	    izz="0.058783"/>
+        <mass value="1.400000"/>
+        <inertia
+            ixx="0.024393" ixy="0.00005" ixz="0.000015"
+	    iyy="0.024541" iyz="0.000205"
+	    izz="0.043817"/>
       </inertial>
       <visual>
         <origin xyz="0 0 0" rpy="0 0 0"/>
         <geometry>
-          <mesh filename="package://gimbalrotor/urdf/beetle/mesh/base_link.dae"/>
+          <mesh filename="package://gimbalrotor/urdf/mesh/beetle_hand_base_link.dae"/>
         </geometry>
       </visual>
@@ -82,14 +82,18 @@
     </xacro:macro>
     ## dummy rotor arms
-    <xacro:dummy_rotor_arm id = "${child1}" x = "0.12129" y="0.12150" z = "0.1185" yaw = "${pi/4.0}"/>
-    <xacro:dummy_rotor_arm id = "${child2}" x = "-0.12129" y="0.12150" z = "0.1185" yaw = "${pi*3.0/4.0}"/>
-    <xacro:dummy_rotor_arm id = "${child3}" x = "-0.12129" y="-0.12150" z = "0.1185" yaw = "${pi*5.0/4.0}"/>
-    <xacro:dummy_rotor_arm id = "${child4}" x = "0.12129" y="-0.12150" z = "0.1185" yaw = "${-pi/4.0}"/>
+    <!-- <xacro:dummy_rotor_arm id = "${child1}" x = "0.12427" y="0.12427" z = "0.11425" yaw = "${pi/4.0}"/> -->
+    <!-- <xacro:dummy_rotor_arm id = "${child2}" x = "-0.12427" y="0.12427" z = "0.11425" yaw = "${pi*3.0/4.0}"/> -->
+    <!-- <xacro:dummy_rotor_arm id = "${child3}" x = "-0.12427" y="-0.12427" z = "0.11425" yaw = "${pi*5.0/4.0}"/> -->
+    <!-- <xacro:dummy_rotor_arm id = "${child4}" x = "0.12427" y="-0.12427" z = "0.11425" yaw = "${pi*7.0/4.0}"/> -->
+    <xacro:dummy_rotor_arm id = "${child1}" x = "0.13427" y="0.13427" z = "0.11425" yaw = "${pi/4.0}"/>
+    <xacro:dummy_rotor_arm id = "${child2}" x = "-0.13427" y="0.13427" z = "0.11425" yaw = "${pi*3.0/4.0}"/>
+    <xacro:dummy_rotor_arm id = "${child3}" x = "-0.13427" y="-0.13427" z = "0.11425" yaw = "${pi*5.0/4.0}"/>
+    <xacro:dummy_rotor_arm id = "${child4}" x = "0.13427" y="-0.13427" z = "0.11425" yaw = "${pi*7.0/4.0}"/>
     ## dummy link for the contact point coordinate
-      <link name="contact_point">
-        <inertial>
-          <origin xyz="0 0 0" rpy="0 0 0"/>
-          <mass value="0.0001"/>
-          <inertia
+    <link name="contact_point">
+      <inertial>
+        <origin xyz="0 0 0" rpy="0 0 0"/>
+        <mass value="0.0001"/>
+        <inertia
               ixx="0.000001" ixy="0.0" ixz="0.0"
               iyy="0.0001" iyz="0.0"
@@ -110,12 +114,13 @@
     <link name="gimbal_link${self}">
       <inertial>
-        <origin xyz="0.0223521 0.0 0.00776312" rpy="0 0 0"/>
-        <mass value="0.15944"/>
-        <inertia
-            ixx="0.00007458" iyy="0.00007325" izz="0.00007756"
-            ixy="0.00000001" ixz="0.00000084" iyz="0.00000001"/>
+        <origin xyz="0.022864 0.0 0.018338" rpy="0 0 0"/>
+        <mass value="0.15000"/>
+        <inertia
+            ixx="0.000063" ixy="0.000003" ixz="0.000000"
+            iyy="0.000057" iyz="0.000000"
+	    izz="0.000063"/>
       </inertial>
       <collision>
-        <origin xyz="0.0 0 0" rpy="0 0 0"/>
+        <origin xyz="0.0 0.0 0.0" rpy="0 0 0"/>
         <geometry>
           <cylinder radius="0.02" length="0.033"/>
@@ -125,5 +130,5 @@
         <origin xyz="0 0 0" rpy="0 0 0"/>
         <geometry>
-          <mesh filename="package://gimbalrotor/urdf/beetle/mesh/rotor_module.dae"/>
+          <mesh filename="package://gimbalrotor/urdf/mesh/beetle_hand_rotor_module.dae"/>
         </geometry>
       </visual>
@@ -199,3 +204,98 @@
     </transmission>
   </xacro:macro>
+  <!-- extra_module -->
+  <xacro:macro name="extra_module" params="name parent *origin *inertial visible:=0 model_url:=0">
+    <joint name="${parent}2${name}" type="fixed">
+      <parent link="${parent}"/>
+      <child link="${name}"/>
+      <xacro:insert_block name="origin" />
+    </joint>
+    <link name="${name}">
+      <xacro:insert_block name="inertial" />
+      <xacro:if value="${visible == 1}">
+        <visual>
+	  <origin rpy="0 0 0" xyz="0 0 0"/>
+          <geometry>
+            <mesh filename="${model_url}" scale="${scale} ${scale} ${scale}"/>
+          </geometry>
+        </visual>
+      </xacro:if>
+    </link>
+  </xacro:macro>
+    ## link
+  <link name="handbase">
+    <inertial>
+      <origin xyz="0.0 0.0 0.0" rpy="0 0 0"/>
+      <mass value="0.00001"/>
+      <inertia
+          ixx="0.00001" iyy="0.00001" izz="0.00001"
+          ixy="0.0" ixz="0.0" iyz="0.0"/>
+    </inertial>
+  </link>
+  <link name="hand">
+    <inertial>
+      <!-- <origin xyz="0.32422 0.004298 0.019803"/> -->
+      <origin xyz="0.19178 0.000005 0.025771"/>
+      <mass value="0.306000"/>
+      <inertia
+  	  ixx="0.0003093" ixy="-0.0002184" ixz="0.0001250"
+    	  iyx="-0.0002184" iyy="0.0023558" iyz="-0.0000268"
+  	  izx="0.0001250" izy="-0.0000268" izz="0.0024254"/>
+      <!-- <inertia -->
+      <!-- 	  ixx="0.000699" ixy="-0.000004" ixz="0.000769" -->
+      <!-- 	  iyy="0.005953" iyz="-0.000005" -->
+      <!-- 	  izz="0.00541"/> -->
+    </inertial>
+    <visual>
+      <origin xyz="0 0 0" rpy="0 0 0"/>
+     <geometry>
+    	<mesh filename="package://beetle/urdf/mesh/Assem_new_complete_s5.STL" scale="0.001 0.001 0.001"/>
+      </geometry>
+    </visual>
+    <collision>
+      <origin xyz="0.236 0.024 0.039" rpy="0 0 0"/>
+      <geometry>
+	<box size="0.471 0.134 0.153"/>
+      </geometry>
+    </collision>
+  </link>
+  <!-- <link name="hand_2"> -->
+  <!--   <inertial> -->
+  <!--     <origin xyz="0.19178 0.000005 0.025771"/> -->
+  <!--     <mass value="0.3900000"/> -->
+  <!--     <inertia -->
+  <!-- 	  ixx="0.000911" ixy="0.001204" ixz="0.000002" -->
+  <!-- 	  iyy="0.009690" iyz="-0.000005" -->
+  <!-- 	  izz="0.010438"/> -->
+  <!--     <!-\- <inertia -\-> -->
+  <!--     <!-\- 	  ixx="0.000699" ixy="-0.000004" ixz="0.000769" -\-> -->
+  <!--     <!-\- 	  iyy="0.005953" iyz="-0.000005" -\-> -->
+  <!--     <!-\- 	  izz="0.00541"/> -\-> -->
+  <!--   </inertial> -->
+  <!--   <visual> -->
+  <!--     <origin xyz="0 0 0" rpy="0 0 0"/> -->
+  <!--     <geometry> -->
+  <!--   	<mesh filename="package://beetle/urdf/mesh/saw.STL" scale="0.1 0.1 0.1"/> -->
+  <!--     </geometry> -->
+  <!--   </visual> -->
+  <!--   <collision> -->
+  <!--     <origin xyz="0.236 0.024 0.039" rpy="0 0 0"/> -->
+  <!--     <geometry> -->
+  <!-- 	<box size="0.471 0.134 0.153"/> -->
+  <!--     </geometry> -->
+  <!--   </collision> -->
+  <!-- </link> -->
+  ## beetle hand joint
+  <joint name="handbase_baselink_joint" type="fixed">
+    <child link="handbase"/>
+    <parent link="base_link"/>
+    <origin xyz="0 0 0" rpy="0 0 0"/>
+    <axis xyz="1 0 0"/>
+  </joint>
+  <joint name="handbase_hand_joint" type="fixed">
+    <child link="hand"/>
+    <parent link="handbase"/>
+    <origin xyz=" 0.05918 0.00052 0.08000" rpy="1.57 0 0"/>
+    <axis xyz="1 0 0"/>
+  </joint>
 </robot>

Commit message: Update gimbalrotor URDF file

File: robots/gimbalrotor/urdf/beetle/gimbalrotor.urdf.xacro (robot description, xacro)
@@ -33,5 +33,5 @@
         <origin xyz="0 0 0" rpy="0 0 0"/>
         <geometry>
-          <mesh filename="package://gimbalrotor/urdf/mesh/beetle_hand_base_link.dae"/>
+          <mesh filename="package://gimbalrotor/urdf/beetle/mesh/base_link.dae"/>
         </geometry>
       </visual>
@@ -130,5 +130,5 @@
         <origin xyz="0 0 0" rpy="0 0 0"/>
         <geometry>
-          <mesh filename="package://gimbalrotor/urdf/mesh/beetle_hand_rotor_module.dae"/>
+          <mesh filename="package://gimbalrotor/urdf/beetle/mesh/rotor_module.dae"/>
         </geometry>
       </visual>
@@ -249,6 +249,6 @@
     <visual>
       <origin xyz="0 0 0" rpy="0 0 0"/>
-     <geometry>
-    	<mesh filename="package://beetle/urdf/mesh/Assem_new_complete_s5.STL" scale="0.001 0.001 0.001"/>
+      <geometry>
+    	<mesh filename="package://gimbalrotor/urdf/beetle/mesh/Assem_new_complete_s5.STL" scale="0.001 0.001 0.001"/>
       </geometry>
     </visual>

Commit message: Edit original beetle urdf to green beetle

File: robots/gimbalrotor/urdf/beetle/gimbalrotor.urdf.xacro (robot description, xacro)
@@ -33,5 +33,5 @@
         <origin xyz="0 0 0" rpy="0 0 0"/>
         <geometry>
-          <mesh filename="package://gimbalrotor/urdf/beetle/mesh/base_link.dae"/>
+          <mesh filename="package://gimbalrotor/urdf/beetle/mesh/beetle_hand_base_link.dae"/>
         </geometry>
       </visual>
@@ -130,5 +130,5 @@
         <origin xyz="0 0 0" rpy="0 0 0"/>
         <geometry>
-          <mesh filename="package://gimbalrotor/urdf/beetle/mesh/rotor_module.dae"/>
+          <mesh filename="package://gimbalrotor/urdf/beetle/mesh/beetle_hand_rotor_module.dae"/>
         </geometry>
       </visual>

Commit message: pochita nopulley testing

File: robots/gimbalrotor/urdf/beetle/gimbalrotor.urdf.xacro (robot description, xacro)
@@ -237,9 +237,9 @@
       <!-- <origin xyz="0.32422 0.004298 0.019803"/> -->
       <origin xyz="0.19178 0.000005 0.025771"/>
-      <mass value="0.306000"/>
+      <mass value="0.323850"/>
       <inertia
-  	  ixx="0.0003093" ixy="-0.0002184" ixz="0.0001250"
-    	  iyx="-0.0002184" iyy="0.0023558" iyz="-0.0000268"
-  	  izx="0.0001250" izy="-0.0000268" izz="0.0024254"/>
+  	  ixx="0.0014298" ixy="-0.0023533" ixz="0.0058413"
+    	  iyx="-0.0023533" iyy="0.0384938" iyz="-0.0004491"
+  	  izx="0.0058413" izy="-0.0004491" izz="0.0374743"/>
       <!-- <inertia -->
       <!-- 	  ixx="0.000699" ixy="-0.000004" ixz="0.000769" -->
@@ -250,5 +250,5 @@
       <origin xyz="0 0 0" rpy="0 0 0"/>
       <geometry>
-    	<mesh filename="package://gimbalrotor/urdf/beetle/mesh/Assem_new_complete_s5.STL" scale="0.001 0.001 0.001"/>
+    	<mesh filename="package://gimbalrotor/urdf/beetle/mesh/fullassem_pochitab_3d.STL" scale="0.001 0.001 0.001"/>
       </geometry>
     </visual>
@@ -296,6 +296,6 @@
     <child link="hand"/>
     <parent link="handbase"/>
-    <origin xyz=" 0.05918 0.00052 0.08000" rpy="1.57 0 0"/>
-    <axis xyz="1 0 0"/>
+    <origin xyz=" 0.05918 0.00052 0.08000" rpy="0 0 0"/>
+    <axis xyz="0 0 0"/>
   </joint>
 </robot>

Commit message: Pochita URDF

File: robots/gimbalrotor/urdf/beetle/gimbalrotor.urdf.xacro (robot description, xacro)
@@ -235,20 +235,15 @@
   <link name="hand">
     <inertial>
-      <!-- <origin xyz="0.32422 0.004298 0.019803"/> -->
       <origin xyz="0.19178 0.000005 0.025771"/>
-      <mass value="0.323850"/>
+      <mass value="0.423690"/>
       <inertia
-  	  ixx="0.0014298" ixy="-0.0023533" ixz="0.0058413"
-    	  iyx="-0.0023533" iyy="0.0384938" iyz="-0.0004491"
-  	  izx="0.0058413" izy="-0.0004491" izz="0.0374743"/>
-      <!-- <inertia -->
-      <!-- 	  ixx="0.000699" ixy="-0.000004" ixz="0.000769" -->
-      <!-- 	  iyy="0.005953" iyz="-0.000005" -->
-      <!-- 	  izz="0.00541"/> -->
+  	  ixx="0.0010323" ixy="-0.0001415" ixz="0.0051142"
+    	  iyx="-0.0001415" iyy="0.0454125" iyz="-0.0000028"
+  	  izx="0.0051142" izy="-0.0000028" izz="0.0446821"/>
     </inertial>
     <visual>
       <origin xyz="0 0 0" rpy="0 0 0"/>
       <geometry>
-    	<mesh filename="package://gimbalrotor/urdf/beetle/mesh/fullassem_pochitab_3d.STL" scale="0.001 0.001 0.001"/>
+    	<mesh filename="package://gimbalrotor/urdf/beetle/mesh/fullassem_pochitab.STL" scale="0.001 0.001 0.001"/>
       </geometry>
     </visual>

Commit message: Hand URDF

File: robots/gimbalrotor/urdf/beetle/gimbalrotor.urdf.xacro (robot description, xacro)
@@ -223,5 +223,5 @@
     </link>
   </xacro:macro>
-    ## link
+  ## link
   <link name="handbase">
     <inertial>
@@ -252,4 +252,31 @@
       <geometry>
 	<box size="0.471 0.134 0.153"/>
+      </geometry>
+    </collision>
+  </link>
+<!-- hand link  -->
+  <link name="hand_2">
+    <inertial>
+      <origin xyz="0.19178 0.000005 0.025771"/>
+      <mass value="0.4100000"/>
+      <inertia
+  	  ixx="0.00092717" ixy="0.00124965" ixz="0.00000526"
+  	  iyy="0.01037553" iyz="0.00000148"
+  	  izz="0.01112688"/>
+      <!-- <inertia -->
+      <!-- 	  ixx="0.000699" ixy="-0.000004" ixz="0.000769" -->
+      <!-- 	  iyy="0.005953" iyz="-0.000005" -->
+      <!-- 	  izz="0.00541"/> -->
+    </inertial>
+    <visual>
+      <origin xyz="0 0 0" rpy="0 0 0"/>
+      <geometry>
+    	<mesh filename="package://gimbalrotor/urdf/beetle/mesh/hand9_handmech_USD.STL" scale="1 1 1"/>
+      </geometry>
+    </visual>
+    <collision>
+      <origin xyz="0.01215 0 0.022" rpy="0 0 0"/>
+      <geometry>
+  	<box size="0.283 0.071 0.118"/>
       </geometry>
     </collision>
@@ -291,6 +318,12 @@
     <child link="hand"/>
     <parent link="handbase"/>
-    <origin xyz=" 0.05918 0.00052 0.08000" rpy="0 0 0"/>
+    <origin xyz="0.05918 0.00052 0.08000" rpy="0 0 0"/>
     <axis xyz="0 0 0"/>
   </joint>
+  <joint name="handbase_hand_joint_2" type="fixed">
+    <child link="hand_2"/>
+    <parent link="handbase"/>
+    <origin xyz="-0.05918 0.00052 0.08000" rpy="0 0 3.1415"/>
+    <axis xyz="1 0 0"/>
+  </joint>
 </robot>

Commit message: [Pochita][URDF] Modified CoG & Inertia

File: robots/gimbalrotor/urdf/beetle/gimbalrotor.urdf.xacro (robot description, xacro)
@@ -235,10 +235,10 @@
   <link name="hand">
     <inertial>
-      <origin xyz="0.19178 0.000005 0.025771"/>
+      <origin xyz="0.316540 0.000030 0.036560"/>
       <mass value="0.423690"/>
       <inertia
   	  ixx="0.0010323" ixy="-0.0001415" ixz="0.0051142"
-    	  iyx="-0.0001415" iyy="0.0454125" iyz="-0.0000028"
-  	  izx="0.0051142" izy="-0.0000028" izz="0.0446821"/>
+    	  iyy="0.0454125" iyz="-0.0000028"
+  	  izz="0.0446821"/>
     </inertial>
     <visual>
@@ -258,10 +258,10 @@
   <link name="hand_2">
     <inertial>
-      <origin xyz="0.19178 0.000005 0.025771"/>
-      <mass value="0.4100000"/>
+      <origin xyz="0.00033 0.056240 0.08802"/>
+      <mass value="0.3100000"/>
       <inertia
-  	  ixx="0.00092282" ixy="0.00105812" ixz="0.00000494"
-  	  iyy="0.01081461" iyz="0.00000144"
-  	  izz="0.01156281"/>
+  	  ixx="0.009713" ixy="-0.00000686" ixz="0.00000217"
+  	  iyy="0.00776047" iyz="0.00266476"
+  	  izz="0.00211585"/>
       <!-- <inertia -->
       <!-- 	  ixx="0.000699" ixy="-0.000004" ixz="0.000769" -->
@@ -272,5 +272,5 @@
       <origin xyz="0 0 0" rpy="0 0 0"/>
       <geometry>
-    	<mesh filename="package://gimbalrotor/urdf/beetle/mesh/hand9_handmech_USD.STL" scale="1 1 1"/>
+    	<mesh filename="package://gimbalrotor/urdf/beetle/mesh/hand9_handmech_USD.STL" scale="0.001 0.001 0.001"/>
       </geometry>
     </visual>
@@ -324,6 +324,6 @@
     <child link="hand_2"/>
     <parent link="handbase"/>
-    <origin xyz="-0.05918 0.00052 0.08000" rpy="0 0 3.1415"/>
-    <axis xyz="1 0 0"/>
+    <origin xyz="-0.05918 0.00052 0.08000" rpy="1.5708 0 4.7124"/>
+    <axis xyz="0 0 0"/>
   </joint>
 </robot>

Commit message: [Pochita][URDF] Hand & Pitch Joint Configuration and Inertia

File: robots/gimbalrotor/urdf/beetle/gimbalrotor.urdf.xacro (robot description, xacro)
@@ -233,12 +233,13 @@
     </inertial>
   </link>
-  <link name="hand">
+  <!-- saw link  -->
+  <link name="saw">
     <inertial>
       <origin xyz="0.316540 0.000030 0.036560"/>
       <mass value="0.423690"/>
       <inertia
-  	  ixx="0.0010323" ixy="-0.0001415" ixz="0.0051142"
-    	  iyy="0.0454125" iyz="-0.0000028"
-  	  izz="0.0446821"/>
+  	  ixx="0.0004659" ixy="-0.0001450" ixz="0.0002106"
+    	  iyy="0.0023921" iyz="-0.0000032"
+  	  izz="0.0022280"/>
     </inertial>
     <visual>
@@ -255,57 +256,50 @@
     </collision>
   </link>
-<!-- hand link  -->
-  <link name="hand_2">
+  <!-- pitch joint fix pipe link  -->
+  <link name="pitch_joint_link">
     <inertial>
-      <origin xyz="0.00033 0.056240 0.08802"/>
-      <mass value="0.3100000"/>
+      <origin xyz="0.16717 0.02381 0.00005"/>
+      <mass value="0.19260"/>
       <inertia
-  	  ixx="0.009713" ixy="-0.00000686" ixz="0.00000217"
-  	  iyy="0.00776047" iyz="0.00266476"
-  	  izz="0.00211585"/>
-      <!-- <inertia -->
-      <!-- 	  ixx="0.000699" ixy="-0.000004" ixz="0.000769" -->
-      <!-- 	  iyy="0.005953" iyz="-0.000005" -->
-      <!-- 	  izz="0.00541"/> -->
+  	  ixx="0.0001889" ixy="0.0000569" ixz="-0.0000002"
+  	  iyy="0.0004543" iyz="0.0000003"
+  	  izz="0.0006006"/>
     </inertial>
     <visual>
       <origin xyz="0 0 0" rpy="0 0 0"/>
       <geometry>
-    	<mesh filename="package://gimbalrotor/urdf/beetle/mesh/hand9_handmech_USD.STL" scale="0.001 0.001 0.001"/>
+    	<mesh filename="package://gimbalrotor/urdf/beetle/mesh/urdf_full_pitchjoint.STL" scale="1 1 1"/>
       </geometry>
     </visual>
     <collision>
-      <origin xyz="0.01215 0 0.022" rpy="0 0 0"/>
-      <geometry>
-  	<box size="0.283 0.071 0.118"/>
+      <origin xyz="0.236 0.024 0" rpy="0 0 0"/>
+      <geometry>
+  	<box size="0.253 0.09 0.038"/>
       </geometry>
     </collision>
   </link>
-  <!-- <link name="hand_2"> -->
-  <!--   <inertial> -->
-  <!--     <origin xyz="0.19178 0.000005 0.025771"/> -->
-  <!--     <mass value="0.3900000"/> -->
-  <!--     <inertia -->
-  <!-- 	  ixx="0.000911" ixy="0.001204" ixz="0.000002" -->
-  <!-- 	  iyy="0.009690" iyz="-0.000005" -->
-  <!-- 	  izz="0.010438"/> -->
-  <!--     <!-\- <inertia -\-> -->
-  <!--     <!-\- 	  ixx="0.000699" ixy="-0.000004" ixz="0.000769" -\-> -->
-  <!--     <!-\- 	  iyy="0.005953" iyz="-0.000005" -\-> -->
-  <!--     <!-\- 	  izz="0.00541"/> -\-> -->
-  <!--   </inertial> -->
-  <!--   <visual> -->
-  <!--     <origin xyz="0 0 0" rpy="0 0 0"/> -->
-  <!--     <geometry> -->
-  <!--   	<mesh filename="package://beetle/urdf/mesh/saw.STL" scale="0.1 0.1 0.1"/> -->
-  <!--     </geometry> -->
-  <!--   </visual> -->
-  <!--   <collision> -->
-  <!--     <origin xyz="0.236 0.024 0.039" rpy="0 0 0"/> -->
-  <!--     <geometry> -->
-  <!-- 	<box size="0.471 0.134 0.153"/> -->
-  <!--     </geometry> -->
-  <!--   </collision> -->
-  <!-- </link> -->
+  <!-- pitch joint hand assem  -->
+  <link name="hand_assem_link">
+    <inertial>
+      <origin xyz="0.09014 0.00038 0.02488"/>
+      <mass value="0.4820000"/>
+      <inertia
+    ixx="0.0008951" ixy="-0.0000298" ixz="0.0006735"
+    iyy="0.0052070" iyz="-0.0000100"
+    izz="0.0045551"/>
+    </inertial>
+    <visual>
+      <origin xyz="0.03658 -0.02307 0.0085" rpy="0 0 0"/>
+      <geometry>
+      <mesh filename="package://gimbalrotor/urdf/beetle/mesh/urdf_full_hand_assem.STL" scale="1 1 1"/>
+      </geometry>
+    </visual>
+    <collision>
+      <origin xyz="0.03658 -0.02307 0.0085" rpy="0 0 0"/>
+      <geometry>
+    <box size="0.5 0.1 0.177"/>
+      </geometry>
+    </collision>
+  </link>
   ## beetle hand joint
   <joint name="handbase_baselink_joint" type="fixed">
@@ -315,15 +309,34 @@
     <axis xyz="1 0 0"/>
   </joint>
-  <joint name="handbase_hand_joint" type="fixed">
-    <child link="hand"/>
+  <joint name="handbase_saw_joint" type="fixed">
+    <child link="saw"/>
     <parent link="handbase"/>
     <origin xyz="0.05918 0.00052 0.08000" rpy="0 0 0"/>
     <axis xyz="0 0 0"/>
   </joint>
-  <joint name="handbase_hand_joint_2" type="fixed">
-    <child link="hand_2"/>
+  <joint name="handbase_pitchpipe_joint" type="fixed">
+    <child link="pitch_joint_link"/>
     <parent link="handbase"/>
-    <origin xyz="-0.05918 0.00052 0.08000" rpy="1.5708 0 4.7124"/>
+    <origin xyz="-0.05918 0.00052 0.08000" rpy="0 0 3.142"/>
     <axis xyz="0 0 0"/>
   </joint>
+  <joint name="pitch_joint" type="revolute">
+    <parent link="pitch_joint_link"/>
+    <child link="hand_assem_link"/>
+    <!-- location of the pitch axis -->
+    <origin xyz="0.22074 0.02307 0" rpy="0 0 0"/>
+    <axis xyz="0 1 0"/>
+    <limit effort="10" velocity="1.0" lower="-1.57" upper="1.57"/>
+    <dynamics damping="0.1" friction="0.01"/>
+  </joint>
+  <transmission name="pitch_joint">
+    <type>transmission_interface/SimpleTransmission</type>
+    <joint name="pitch_joint">
+      <hardwareInterface>hardware_interface/EffortJointInterface</hardwareInterface>
+    </joint>
+    <actuator name="pitch_joint">
+      <hardwareInterface>hardware_interface/EffortJointInterface</hardwareInterface>
+      <mechanicalReduction>1</mechanicalReduction>
+    </actuator>
+  </transmission>
 </robot>

Commit message: [Beetle][saw] Workaroud to read joint state from servos connected to another Spinal.

File: robots/gimbalrotor/urdf/beetle/gimbalrotor.urdf.xacro (robot description, xacro)
@@ -330,4 +330,22 @@
     <dynamics damping="0.1" friction="0.01"/>
   </joint>
+  <joint name="wire_joint" type="revolute">
+    <parent link="base_link"/>
+    <child link="virtual_wire"/>
+    <limit effort="10" velocity="1.0" lower="-1.57" upper="1.57"/>
+    <dynamics damping="0.1" friction="0.01"/>
+    <origin rpy="0 0 0" xyz="0 0 0"/>
+    <axis xyz="0 0 1"/>
+  </joint>
+  <link name="virtual_wire">
+    <inertial>
+      <origin xyz="0 0 0" rpy="0 0 0"/>
+      <mass value="0.00001"/>
+      <inertia
+          ixx="0.00001" ixy="0.0" ixz="0.0"
+          iyy="0.00001" iyz="0.0"
+          izz="0.00001"/>
+    </inertial>
+  </link>
   <transmission name="pitch_joint">
     <type>transmission_interface/SimpleTransmission</type>
@@ -340,3 +358,13 @@
     </actuator>
   </transmission>
+  <transmission name="wire_joint">
+    <type>transmission_interface/SimpleTransmission</type>
+    <joint name="wire_joint">
+      <hardwareInterface>hardware_interface/EffortJointInterface</hardwareInterface>
+    </joint>
+    <actuator name="wire_joint">
+      <hardwareInterface>hardware_interface/EffortJointInterface</hardwareInterface>
+      <mechanicalReduction>1</mechanicalReduction>
+    </actuator>
+  </transmission>
 </robot>

Commit message: [Pochita][Perching] Pitch Perching Configuration & Adjusted Pitch Joint URDF

File: robots/gimbalrotor/urdf/beetle/gimbalrotor.urdf.xacro (robot description, xacro)
@@ -290,5 +290,5 @@
     </inertial>
     <visual>
-      <origin xyz="0.03658 -0.02307 0.0085" rpy="0 0 0"/>
+      <origin xyz="0.03658 -0.02932 0.0085" rpy="0 0 0"/>
       <geometry>
       <mesh filename="package://gimbalrotor/urdf/beetle/mesh/urdf_full_hand_assem.STL" scale="1 1 1"/>
@@ -325,5 +325,5 @@
     <child link="hand_assem_link"/>
     <!-- location of the pitch axis -->
-    <origin xyz="0.22074 0.02307 0" rpy="0 0 0"/>
+    <origin xyz="0.22074 0.02932 0" rpy="0 0 0"/>  <!-- 0.02932 is pulley origin -->
     <axis xyz="0 1 0"/>
     <limit effort="10" velocity="1.0" lower="-1.57" upper="1.57"/>
