Commit message: [Pochita] Multilink behaviour: changed "model" && "navigation"

File: robots/gimbalrotor/urdf/beetle/gimbalrotor.urdf.xacro (robot description, xacro)
@@ -327,6 +327,6 @@
     <origin xyz="0.22074 0.02932 0" rpy="0 0 0"/>  <!-- 0.02932 is pulley origin -->
     <axis xyz="0 1 0"/>
-    <limit effort="10" velocity="1.0" lower="-1.57" upper="1.57"/>
-    <dynamics damping="0.1" friction="0.01"/>
+    <limit effort="10" velocity="0.1" lower="-1.57" upper="1.57"/>
+    <dynamics damping="0.9" friction="0.05"/>
   </joint>
   <joint name="wire_joint" type="revolute">

Commit message: [All] Changed from multilink back to normal gimbalrotor

File: robots/gimbalrotor/urdf/beetle/gimbalrotor.urdf.xacro (robot description, xacro)
@@ -269,5 +269,5 @@
       <origin xyz="0 0 0" rpy="0 0 0"/>
       <geometry>
-    	<mesh filename="package://gimbalrotor/urdf/beetle/mesh/urdf_full_pitchjoint.STL" scale="1 1 1"/>
+    	<mesh filename="package://gimbalrotor/urdf/beetle/mesh/passive_perching_hand.STL" scale="1 1 1"/>
       </geometry>
     </visual>
@@ -280,5 +280,5 @@
   </link>
   <!-- pitch joint hand assem  -->
-  <link name="hand_assem_link">
+  <!-- <link name="hand_assem_link">
     <inertial>
       <origin xyz="0.09014 0.00038 0.02488"/>
@@ -301,5 +301,5 @@
       </geometry>
     </collision>
-  </link>
+  </link>   -->
   ## beetle hand joint
   <joint name="handbase_baselink_joint" type="fixed">
@@ -321,50 +321,3 @@
     <axis xyz="0 0 0"/>
   </joint>
-  <joint name="pitch_joint" type="revolute">
-    <parent link="pitch_joint_link"/>
-    <child link="hand_assem_link"/>
-    <!-- location of the pitch axis -->
-    <origin xyz="0.22074 0.02932 0" rpy="0 0 0"/>  <!-- 0.02932 is pulley origin -->
-    <axis xyz="0 1 0"/>
-    <limit effort="10" velocity="0.1" lower="-1.57" upper="1.57"/>
-    <dynamics damping="0.9" friction="0.05"/>
-  </joint>
-  <joint name="wire_joint" type="revolute">
-    <parent link="base_link"/>
-    <child link="virtual_wire"/>
-    <limit effort="10" velocity="1.0" lower="-1.57" upper="1.57"/>
-    <dynamics damping="0.1" friction="0.01"/>
-    <origin rpy="0 0 0" xyz="0 0 0"/>
-    <axis xyz="0 0 1"/>
-  </joint>
-  <link name="virtual_wire">
-    <inertial>
-      <origin xyz="0 0 0" rpy="0 0 0"/>
-      <mass value="0.00001"/>
-      <inertia
-          ixx="0.00001" ixy="0.0" ixz="0.0"
-          iyy="0.00001" iyz="0.0"
-          izz="0.00001"/>
-    </inertial>
-  </link>
-  <transmission name="pitch_joint">
-    <type>transmission_interface/SimpleTransmission</type>
-    <joint name="pitch_joint">
-      <hardwareInterface>hardware_interface/EffortJointInterface</hardwareInterface>
-    </joint>
-    <actuator name="pitch_joint">
-      <hardwareInterface>hardware_interface/EffortJointInterface</hardwareInterface>
-      <mechanicalReduction>1</mechanicalReduction>
-    </actuator>
-  </transmission>
-  <transmission name="wire_joint">
-    <type>transmission_interface/SimpleTransmission</type>
-    <joint name="wire_joint">
-      <hardwareInterface>hardware_interface/EffortJointInterface</hardwareInterface>
-    </joint>
-    <actuator name="wire_joint">
-      <hardwareInterface>hardware_interface/EffortJointInterface</hardwareInterface>
-      <mechanicalReduction>1</mechanicalReduction>
-    </actuator>
-  </transmission>
 </robot>

Commit message: [URDF] Inertia changed

File: robots/gimbalrotor/urdf/beetle/gimbalrotor.urdf.xacro (robot description, xacro)
@@ -2,4 +2,6 @@
 <robot
     xmlns:xacro="http://www.ros.org/wiki/xacro" name="gimbalrotor_link" >
+  <xacro:arg name="use_saw" default="true"/>
+  <xacro:arg name="use_hand" default="true"/>
   <xacro:macro name="gimbalrotor_center_link" params="child1 child2 child3 child4">
     ## dummy
@@ -91,20 +93,20 @@
     <xacro:dummy_rotor_arm id = "${child4}" x = "0.13427" y="-0.13427" z = "0.11425" yaw = "${pi*7.0/4.0}"/>
     ## dummy link for the contact point coordinate
-    <link name="contact_point">
-      <inertial>
-        <origin xyz="0 0 0" rpy="0 0 0"/>
-        <mass value="0.0001"/>
-        <inertia
-              ixx="0.000001" ixy="0.0" ixz="0.0"
-              iyy="0.0001" iyz="0.0"
-              izz="0.0001"/>
-        </inertial>
-      </link>
-      <joint name="cp_base_joint" type="fixed">
-        <parent link="base_link"/>
-        <child link="contact_point"/>
-        <origin rpy="0 0 0" xyz="0.26 0 0"/>
-        <axis xyz="0 0 1"/>
-      </joint>
+    <!-- <link name="contact_point"> -->
+    <!--   <inertial> -->
+    <!--     <origin xyz="0 0 0" rpy="0 0 0"/> -->
+    <!--     <mass value="0.0001"/> -->
+    <!--     <inertia -->
+    <!--           ixx="0.000001" ixy="0.0" ixz="0.0" -->
+    <!--           iyy="0.0001" iyz="0.0" -->
+    <!--           izz="0.0001"/> -->
+    <!--     </inertial> -->
+    <!--   </link> -->
+    <!--   <joint name="cp_base_joint" type="fixed"> -->
+    <!--     <parent link="base_link"/> -->
+    <!--     <child link="contact_point"/> -->
+    <!--     <origin rpy="0 0 0" xyz="0.26 0 0"/> -->
+    <!--     <axis xyz="0 0 1"/> -->
+    <!--   </joint> -->
     <xacro:friction self="base_link"/>
   </xacro:macro>
@@ -205,22 +207,22 @@
   </xacro:macro>
   <!-- extra_module -->
-  <xacro:macro name="extra_module" params="name parent *origin *inertial visible:=0 model_url:=0">
-    <joint name="${parent}2${name}" type="fixed">
-      <parent link="${parent}"/>
-      <child link="${name}"/>
-      <xacro:insert_block name="origin" />
-    </joint>
-    <link name="${name}">
-      <xacro:insert_block name="inertial" />
-      <xacro:if value="${visible == 1}">
-        <visual>
-	  <origin rpy="0 0 0" xyz="0 0 0"/>
-          <geometry>
-            <mesh filename="${model_url}" scale="${scale} ${scale} ${scale}"/>
-          </geometry>
-        </visual>
-      </xacro:if>
-    </link>
-  </xacro:macro>
+  <!-- <xacro:macro name="extra_module" params="name parent *origin *inertial visible:=0 model_url:=0"> -->
+  <!--   <joint name="${parent}2${name}" type="fixed"> -->
+  <!--     <parent link="${parent}"/> -->
+  <!--     <child link="${name}"/> -->
+  <!--     <xacro:insert_block name="origin" /> -->
+  <!--   </joint> -->
+  <!--   <link name="${name}"> -->
+  <!--     <xacro:insert_block name="inertial" /> -->
+  <!--     <xacro:if value="${visible == 1}"> -->
+  <!--       <visual> -->
+  <!-- 	  <origin rpy="0 0 0" xyz="0 0 0"/> -->
+  <!--         <geometry> -->
+  <!--           <mesh filename="${model_url}" scale="${scale} ${scale} ${scale}"/> -->
+  <!--         </geometry> -->
+  <!--       </visual> -->
+  <!--     </xacro:if> -->
+  <!--   </link> -->
+  <!-- </xacro:macro> -->
   ## link
   <link name="handbase">
@@ -233,73 +235,54 @@
     </inertial>
   </link>
-  <!-- saw link  -->
-  <link name="saw">
-    <inertial>
-      <origin xyz="0.316540 0.000030 0.036560"/>
-      <mass value="0.423690"/>
-      <inertia
-  	  ixx="0.0004659" ixy="-0.0001450" ixz="0.0002106"
-    	  iyy="0.0023921" iyz="-0.0000032"
-  	  izz="0.0022280"/>
-    </inertial>
-    <visual>
-      <origin xyz="0 0 0" rpy="0 0 0"/>
-      <geometry>
-    	<mesh filename="package://gimbalrotor/urdf/beetle/mesh/fullassem_pochitab.STL" scale="0.001 0.001 0.001"/>
-      </geometry>
-    </visual>
-    <collision>
-      <origin xyz="0.236 0.024 0.039" rpy="0 0 0"/>
-      <geometry>
-	<box size="0.471 0.134 0.153"/>
-      </geometry>
-    </collision>
-  </link>
-  <!-- pitch joint fix pipe link  -->
-  <link name="pitch_joint_link">
-    <inertial>
-      <origin xyz="0.16717 0.02381 0.00005"/>
-      <mass value="0.19260"/>
-      <inertia
-  	  ixx="0.0001889" ixy="0.0000569" ixz="-0.0000002"
-  	  iyy="0.0004543" iyz="0.0000003"
-  	  izz="0.0006006"/>
-    </inertial>
-    <visual>
-      <origin xyz="0 0 0" rpy="0 0 0"/>
-      <geometry>
-    	<mesh filename="package://gimbalrotor/urdf/beetle/mesh/passive_perching_hand.STL" scale="1 1 1"/>
-      </geometry>
-    </visual>
-    <collision>
-      <origin xyz="0.236 0.024 0" rpy="0 0 0"/>
-      <geometry>
-  	<box size="0.253 0.09 0.038"/>
-      </geometry>
-    </collision>
-  </link>
-  <!-- pitch joint hand assem  -->
-  <!-- <link name="hand_assem_link">
-    <inertial>
-      <origin xyz="0.09014 0.00038 0.02488"/>
-      <mass value="0.4820000"/>
-      <inertia
-    ixx="0.0008951" ixy="-0.0000298" ixz="0.0006735"
-    iyy="0.0052070" iyz="-0.0000100"
-    izz="0.0045551"/>
-    </inertial>
-    <visual>
-      <origin xyz="0.03658 -0.02932 0.0085" rpy="0 0 0"/>
-      <geometry>
-      <mesh filename="package://gimbalrotor/urdf/beetle/mesh/urdf_full_hand_assem.STL" scale="1 1 1"/>
-      </geometry>
-    </visual>
-    <collision>
-      <origin xyz="0.03658 -0.02307 0.0085" rpy="0 0 0"/>
-      <geometry>
-    <box size="0.5 0.1 0.177"/>
-      </geometry>
-    </collision>
-  </link>   -->
+  <xacro:if value="$(arg use_saw)">
+    <!-- saw link  -->
+    <link name="saw">
+      <inertial>
+	<origin xyz="0.31654 0.00003 0.03656"/>
+	<mass value="0.423690"/>
+	<inertia
+	    ixx="0.0004659" ixy="-0.00014505" ixz="0.0002106"
+	    iyy="0.0023921" iyz="-0.00000324"
+	    izz="0.00222804"/>
+      </inertial>
+      <visual>
+	<origin xyz="0 0 0" rpy="0 0 0"/>
+	<geometry>
+    	  <mesh filename="package://gimbalrotor/urdf/beetle/mesh/fullassem_pochitab.STL" scale="0.001 0.001 0.001"/>
+	</geometry>
+      </visual>
+      <collision>
+	<origin xyz="0.236 0.024 0.039" rpy="0 0 0"/>
+	<geometry>
+	  <box size="0.471 0.134 0.153"/>
+	</geometry>
+      </collision>
+    </link>
+  </xacro:if>
+  <xacro:if value="$(arg use_hand)">
+    ## passive hand link
+    <link name="passive_hand_link">
+      <inertial>
+	<origin xyz="0.18069 0.00008 0.00001"/>
+	<mass value="0.110"/>
+	<inertia
+	    ixx="0.0000221" ixy="0.0000001" ixz="-0.00000004"
+	    iyy="0.0005956" iyz="0.000000006"
+	    izz="0.0005915"/>
+      </inertial>
+      <visual>
+	<origin xyz="0 0 0" rpy="0 0 0"/>
+	<geometry>
+    	  <mesh filename="package://gimbalrotor/urdf/beetle/mesh/passive_perching_hand.STL" scale="1 1 1"/>
+	</geometry>
+      </visual>
+      <collision>
+	<origin xyz="0.236 0.024 0" rpy="0 0 0"/>
+	<geometry>
+	  <box size="0.253 0.09 0.038"/>
+	</geometry>
+      </collision>
+    </link>
+  </xacro:if>
   ## beetle hand joint
   <joint name="handbase_baselink_joint" type="fixed">
@@ -309,15 +292,19 @@
     <axis xyz="1 0 0"/>
   </joint>
-  <joint name="handbase_saw_joint" type="fixed">
-    <child link="saw"/>
-    <parent link="handbase"/>
-    <origin xyz="0.05918 0.00052 0.08000" rpy="0 0 0"/>
-    <axis xyz="0 0 0"/>
-  </joint>
-  <joint name="handbase_pitchpipe_joint" type="fixed">
-    <child link="pitch_joint_link"/>
-    <parent link="handbase"/>
-    <origin xyz="-0.05918 0.00052 0.08000" rpy="0 0 3.142"/>
-    <axis xyz="0 0 0"/>
-  </joint>
+  <xacro:if value="$(arg use_saw)">
+    <joint name="handbase_saw_joint" type="fixed">
+      <child link="saw"/>
+      <parent link="handbase"/>
+      <origin xyz="0.05918 0.00052 0.08000" rpy="0 0 0"/>
+      <axis xyz="0 0 0"/>
+    </joint>
+  </xacro:if>
+  <xacro:if value="$(arg use_hand)">
+    <joint name="handbase_pitchpipe_joint" type="fixed">
+      <child link="passive_hand_link"/>
+      <parent link="handbase"/>
+      <origin xyz="-0.05918 0.00052 0.08000" rpy="0 0 3.142"/>
+      <axis xyz="0 0 0"/>
+    </joint>
+  </xacro:if>
 </robot>

Commit message: [URDF] according to SW config, but cannot takeoff

File: robots/gimbalrotor/urdf/beetle/gimbalrotor.urdf.xacro (robot description, xacro)
@@ -235,10 +235,10 @@
   <link name="hand">
     <inertial>
-      <origin xyz="0.19178 0.000005 0.025771"/>
+      <origin xyz="0.31654 0.00003 0.03656"/>
       <mass value="0.423690"/>
       <inertia
-  	  ixx="0.0010323" ixy="-0.0001415" ixz="0.0051142"
-    	  iyx="-0.0001415" iyy="0.0454125" iyz="-0.0000028"
-  	  izx="0.0051142" izy="-0.0000028" izz="0.0446821"/>
+  	  ixx="0.0004659" ixy="-0.0001450" ixz="0.0002106"
+    	  iyy="0.0023921" iyz="-0.0000032"
+  	  izz="0.0022280"/>
     </inertial>
     <visual>

Commit message: [URDF] Updated URDF & PID

File: robots/gimbalrotor/urdf/beetle/gimbalrotor.urdf.xacro (robot description, xacro)
@@ -233,26 +233,26 @@
     </inertial>
   </link>
-  <link name="hand">
-    <inertial>
-      <origin xyz="0.31654 0.00003 0.03656"/>
-      <mass value="0.423690"/>
-      <inertia
-  	  ixx="0.0004659" ixy="-0.0001450" ixz="0.0002106"
-    	  iyy="0.0023921" iyz="-0.0000032"
-  	  izz="0.0022280"/>
-    </inertial>
-    <visual>
-      <origin xyz="0 0 0" rpy="0 0 0"/>
-      <geometry>
-    	<mesh filename="package://gimbalrotor/urdf/beetle/mesh/fullassem_pochitab.STL" scale="0.001 0.001 0.001"/>
-      </geometry>
-    </visual>
-    <collision>
-      <origin xyz="0.236 0.024 0.039" rpy="0 0 0"/>
-      <geometry>
-	<box size="0.471 0.134 0.153"/>
-      </geometry>
-    </collision>
-  </link>
+  <!-- <link name="hand"> -->
+  <!--   <inertial> -->
+  <!--     <origin xyz="0.31654 0.00003 0.03656"/> -->
+  <!--     <mass value="0.423690"/> -->
+  <!--     <inertia -->
+  <!-- 	  ixx="0.0004659" ixy="-0.0001450" ixz="0.0002106" -->
+  <!--   	  iyy="0.0023921" iyz="-0.0000032" -->
+  <!-- 	  izz="0.0022280"/> -->
+  <!--   </inertial> -->
+  <!--   <visual> -->
+  <!--     <origin xyz="0 0 0" rpy="0 0 0"/> -->
+  <!--     <geometry> -->
+  <!--   	<mesh filename="package://gimbalrotor/urdf/beetle/mesh/fullassem_pochitab.STL" scale="0.001 0.001 0.001"/> -->
+  <!--     </geometry> -->
+  <!--   </visual> -->
+  <!--   <collision> -->
+  <!--     <origin xyz="0.236 0.024 0.039" rpy="0 0 0"/> -->
+  <!--     <geometry> -->
+  <!-- 	<box size="0.471 0.134 0.153"/> -->
+  <!--     </geometry> -->
+  <!--   </collision> -->
+  <!-- </link> -->
   <!-- <link name="hand_2"> -->
   <!--   <inertial> -->
@@ -288,9 +288,9 @@
     <axis xyz="1 0 0"/>
   </joint>
-  <joint name="handbase_hand_joint" type="fixed">
-    <child link="hand"/>
-    <parent link="handbase"/>
-    <origin xyz=" 0.05918 0.00052 0.08000" rpy="0 0 0"/>
-    <axis xyz="0 0 0"/>
-  </joint>
+  <!-- <joint name="handbase_hand_joint" type="fixed"> -->
+  <!--   <child link="hand"/> -->
+  <!--   <parent link="handbase"/> -->
+  <!--   <origin xyz=" 0.05918 0.00052 0.08000" rpy="0 0 0"/> -->
+  <!--   <axis xyz="0 0 0"/> -->
+  <!-- </joint> -->
 </robot>

Commit message: [Sync] push to remote

File: robots/gimbalrotor/urdf/beetle/gimbalrotor.urdf.xacro (robot description, xacro)
@@ -223,14 +223,14 @@
     </link>
   </xacro:macro>
-    ## link
-  <link name="handbase">
-    <inertial>
-      <origin xyz="0.0 0.0 0.0" rpy="0 0 0"/>
-      <mass value="0.00001"/>
-      <inertia
-          ixx="0.00001" iyy="0.00001" izz="0.00001"
-          ixy="0.0" ixz="0.0" iyz="0.0"/>
-    </inertial>
-  </link>
+  <!--   ## link -->
+  <!-- <link name="handbase"> -->
+  <!--   <inertial> -->
+  <!--     <origin xyz="0.0 0.0 0.0" rpy="0 0 0"/> -->
+  <!--     <mass value="0.00001"/> -->
+  <!--     <inertia -->
+  <!--         ixx="0.00001" iyy="0.00001" izz="0.00001" -->
+  <!--         ixy="0.0" ixz="0.0" iyz="0.0"/> -->
+  <!--   </inertial> -->
+  <!-- </link> -->
   <!-- <link name="hand"> -->
   <!--   <inertial> -->
@@ -281,11 +281,11 @@
   <!--   </collision> -->
   <!-- </link> -->
-  ## beetle hand joint
-  <joint name="handbase_baselink_joint" type="fixed">
-    <child link="handbase"/>
-    <parent link="base_link"/>
-    <origin xyz="0 0 0" rpy="0 0 0"/>
-    <axis xyz="1 0 0"/>
-  </joint>
+  <!-- ## beetle hand joint -->
+  <!-- <joint name="handbase_baselink_joint" type="fixed"> -->
+  <!--   <child link="handbase"/> -->
+  <!--   <parent link="base_link"/> -->
+  <!--   <origin xyz="0 0 0" rpy="0 0 0"/> -->
+  <!--   <axis xyz="1 0 0"/> -->
+  <!-- </joint> -->
   <!-- <joint name="handbase_hand_joint" type="fixed"> -->
   <!--   <child link="hand"/> -->

Commit message: [Changes] Can fly normally

File: robots/gimbalrotor/urdf/beetle/gimbalrotor.urdf.xacro (robot description, xacro)
@@ -91,20 +91,20 @@
     <xacro:dummy_rotor_arm id = "${child4}" x = "0.13427" y="-0.13427" z = "0.11425" yaw = "${pi*7.0/4.0}"/>
     ## dummy link for the contact point coordinate
-    <link name="contact_point">
-      <inertial>
-        <origin xyz="0 0 0" rpy="0 0 0"/>
-        <mass value="0.0001"/>
-        <inertia
-              ixx="0.000001" ixy="0.0" ixz="0.0"
-              iyy="0.0001" iyz="0.0"
-              izz="0.0001"/>
-        </inertial>
-      </link>
-      <joint name="cp_base_joint" type="fixed">
-        <parent link="base_link"/>
-        <child link="contact_point"/>
-        <origin rpy="0 0 0" xyz="0.26 0 0"/>
-        <axis xyz="0 0 1"/>
-      </joint>
+    <!-- <link name="contact_point"> -->
+    <!--   <inertial> -->
+    <!--     <origin xyz="0 0 0" rpy="0 0 0"/> -->
+    <!--     <mass value="0.0001"/> -->
+    <!--     <inertia -->
+    <!--           ixx="0.000001" ixy="0.0" ixz="0.0" -->
+    <!--           iyy="0.0001" iyz="0.0" -->
+    <!--           izz="0.0001"/> -->
+    <!--     </inertial> -->
+    <!--   </link> -->
+    <!--   <joint name="cp_base_joint" type="fixed"> -->
+    <!--     <parent link="base_link"/> -->
+    <!--     <child link="contact_point"/> -->
+    <!--     <origin rpy="0 0 0" xyz="0.26 0 0"/> -->
+    <!--     <axis xyz="0 0 1"/> -->
+    <!--   </joint> -->
     <xacro:friction self="base_link"/>
   </xacro:macro>
@@ -205,22 +205,22 @@
   </xacro:macro>
   <!-- extra_module -->
-  <xacro:macro name="extra_module" params="name parent *origin *inertial visible:=0 model_url:=0">
-    <joint name="${parent}2${name}" type="fixed">
-      <parent link="${parent}"/>
-      <child link="${name}"/>
-      <xacro:insert_block name="origin" />
-    </joint>
-    <link name="${name}">
-      <xacro:insert_block name="inertial" />
-      <xacro:if value="${visible == 1}">
-        <visual>
-	  <origin rpy="0 0 0" xyz="0 0 0"/>
-          <geometry>
-            <mesh filename="${model_url}" scale="${scale} ${scale} ${scale}"/>
-          </geometry>
-        </visual>
-      </xacro:if>
-    </link>
-  </xacro:macro>
+  <!-- <xacro:macro name="extra_module" params="name parent *origin *inertial visible:=0 model_url:=0"> -->
+  <!--   <joint name="${parent}2${name}" type="fixed"> -->
+  <!--     <parent link="${parent}"/> -->
+  <!--     <child link="${name}"/> -->
+  <!--     <xacro:insert_block name="origin" /> -->
+  <!--   </joint> -->
+  <!--   <link name="${name}"> -->
+  <!--     <xacro:insert_block name="inertial" /> -->
+  <!--     <xacro:if value="${visible == 1}"> -->
+  <!--       <visual> -->
+  <!-- 	  <origin rpy="0 0 0" xyz="0 0 0"/> -->
+  <!--         <geometry> -->
+  <!--           <mesh filename="${model_url}" scale="${scale} ${scale} ${scale}"/> -->
+  <!--         </geometry> -->
+  <!--       </visual> -->
+  <!--     </xacro:if> -->
+  <!--   </link> -->
+  <!-- </xacro:macro> -->
   <!--   ## link -->
   <!-- <link name="handbase"> -->

Commit message: [URDF] Changed to 27.5

File: robots/gimbalrotor/urdf/beetle/gimbalrotor.urdf.xacro (robot description, xacro)
@@ -264,15 +264,15 @@
     <link name="passive_hand_link">
       <inertial>
-	<origin xyz="0.18069 0.00008 0.00001"/>
-	<mass value="0.110"/>
+	<origin xyz="0.16829 0.00007 0.00007"/>
+	<mass value="0.150"/>
 	<inertia
-	    ixx="0.0000221" ixy="0.0000001" ixz="-0.00000004"
-	    iyy="0.0005956" iyz="0.000000006"
-	    izz="0.0005915"/>
+	    ixx="0.0000323" ixy="0.0000003" ixz="-0.0000014"
+	    iyy="0.0010134" iyz="0.000000006"
+	    izz="0.0010082"/>
       </inertial>
       <visual>
 	<origin xyz="0 0 0" rpy="0 0 0"/>
 	<geometry>
-    	  <mesh filename="package://gimbalrotor/urdf/beetle/mesh/passive_perching_hand.STL" scale="1 1 1"/>
+    	  <mesh filename="package://gimbalrotor/urdf/beetle/mesh/passive_perching_hand_275.STL" scale="1 1 1"/>
 	</geometry>
       </visual>

Commit message: [URDF] Changed to 60

File: robots/gimbalrotor/urdf/beetle/gimbalrotor.urdf.xacro (robot description, xacro)
@@ -2,5 +2,5 @@
 <robot
     xmlns:xacro="http://www.ros.org/wiki/xacro" name="gimbalrotor_link" >
-  <xacro:arg name="use_saw" default="true"/>
+  <xacro:arg name="use_saw" default="false"/>
   <xacro:arg name="use_hand" default="true"/>
   <xacro:macro name="gimbalrotor_center_link" params="child1 child2 child3 child4">
@@ -264,5 +264,5 @@
     <link name="passive_hand_link">
       <inertial>
-	<origin xyz="0.16829 0.00007 0.00007"/>
+	<origin xyz="0.16829 0.00007 0.00007"/> <!-- 27.5 -->
 	<mass value="0.150"/>
 	<inertia
@@ -270,4 +270,10 @@
 	    iyy="0.0010134" iyz="0.000000006"
 	    izz="0.0010082"/>
+	<!-- <origin xyz="0.20096 0.00005 0.00005"/> <!-\- 60 -\->  -->
+	<!-- <mass value="0.210"/> -->
+	<!-- <inertia -->
+	<!--     ixx="0.0000946" ixy="-0.00000006" ixz="-0.0000018" -->
+	<!--     iyy="0.0017155" iyz="0.000000007" -->
+	<!--     izz="0.0016576"/> -->
       </inertial>
       <visual>

Commit message: [Perching Config] 1. Improve perching radius config 2. Improve trigger of perching nav and perching impedance

File: robots/gimbalrotor/urdf/beetle/gimbalrotor.urdf.xacro (robot description, xacro)
@@ -264,21 +264,21 @@
     <link name="passive_hand_link">
       <inertial>
-	<origin xyz="0.16829 0.00007 0.00007"/> <!-- 27.5 -->
-	<mass value="0.150"/>
+	<!-- <origin xyz="0.16829 0.00007 0.00007"/> <!-\- 26 or 27.5 -\-> -->
+	<!-- <mass value="0.150"/> -->
+	<!-- <inertia -->
+	<!--     ixx="0.0000323" ixy="0.0000003" ixz="-0.0000014" -->
+	<!--     iyy="0.0010134" iyz="0.000000006" -->
+	<!--     izz="0.0010082"/> -->
+	<origin xyz="0.20096 0.00005 0.00005"/> <!-- 60 or 63 -->
+	<mass value="0.210"/>
 	<inertia
-	    ixx="0.0000323" ixy="0.0000003" ixz="-0.0000014"
-	    iyy="0.0010134" iyz="0.000000006"
-	    izz="0.0010082"/>
-	<!-- <origin xyz="0.20096 0.00005 0.00005"/> <!-\- 60 -\->  -->
-	<!-- <mass value="0.210"/> -->
-	<!-- <inertia -->
-	<!--     ixx="0.0000946" ixy="-0.00000006" ixz="-0.0000018" -->
-	<!--     iyy="0.0017155" iyz="0.000000007" -->
-	<!--     izz="0.0016576"/> -->
+	    ixx="0.0000946" ixy="-0.00000006" ixz="-0.0000018"
+	    iyy="0.0017155" iyz="0.000000007"
+	    izz="0.0016576"/>
       </inertial>
       <visual>
 	<origin xyz="0 0 0" rpy="0 0 0"/>
 	<geometry>
-    	  <mesh filename="package://gimbalrotor/urdf/beetle/mesh/passive_perching_hand_275.STL" scale="1 1 1"/>
+    	  <mesh filename="package://gimbalrotor/urdf/beetle/mesh/passive_perching_hand_630.STL" scale="1 1 1"/>
 	</geometry>
       </visual>
