Commit message: [URDF] Adjusted inertia for beetle 4.1

File: robots/gimbalrotor/urdf/beetle/gimbalrotor.urdf.xacro (robot description, xacro)
@@ -25,21 +25,21 @@
     <link name="base_link">
       <inertial>
-        <origin xyz="0.000169 0.002346 0.106123" rpy="0 0 0"/>
-        <mass value="1.400000"/>
-        <inertia
-            ixx="0.024393" ixy="0.00005" ixz="0.000015"
-	    iyy="0.024541" iyz="0.000205"
-	    izz="0.043817"/>
-      </inertial>
-      <visual>
-        <origin xyz="0 0 0" rpy="0 0 0"/>
-        <geometry>
-          <mesh filename="package://gimbalrotor/urdf/beetle/mesh/beetle_hand_base_link.dae"/>
-        </geometry>
-      </visual>
-      <collision>
-        <origin xyz="0 0 0.1065" rpy="0 0 0"/>
-        <geometry>
-          <box size="0.518 0.518 0.213"/>
+        <origin xyz="0.00193 0.00159 0.06156" rpy="0 0 0"/>  #################<!-- Changed -->
+        <mass value="1.444000"/>  #################<!-- Changed -->
+        <inertia
+          ixx="0.0368599" ixy="-0.0000221" ixz="0.0002913"
+	        iyy="0.0367152" iyz="-0.00007901"
+	        izz="0.0663418"/>
+      </inertial>  #################<!-- Changed -->
+      <visual>
+        <origin xyz="0 0 0" rpy="0 0 0"/>
+        <geometry>
+          <mesh filename="package://gimbalrotor/urdf/beetle/mesh/base_module_incenter.STL" scale="0.001 0.001 0.001"/>  #################<!-- Changed -->
+        </geometry>
+      </visual>
+      <collision>
+        <origin xyz="0 0 0.0575" rpy="0 0 0"/>
+        <geometry>
+          <box size="0.518 0.518 0.241"/>
         </geometry>
       </collision>
@@ -59,5 +59,5 @@
       <child link="fc"/>
       <parent link="base_link"/>
-      <origin rpy="0 0 0" xyz="0 0 0.12947"/>
+      <origin rpy="0 0 0" xyz="0 0 0.06927"/>  #################<!-- Changed -->
       <axis xyz="0 0 1"/>
     </joint>
@@ -83,30 +83,8 @@
       </joint>
     </xacro:macro>
-    ## dummy rotor arms
-    <!-- <xacro:dummy_rotor_arm id = "${child1}" x = "0.12427" y="0.12427" z = "0.11425" yaw = "${pi/4.0}"/> -->
-    <!-- <xacro:dummy_rotor_arm id = "${child2}" x = "-0.12427" y="0.12427" z = "0.11425" yaw = "${pi*3.0/4.0}"/> -->
-    <!-- <xacro:dummy_rotor_arm id = "${child3}" x = "-0.12427" y="-0.12427" z = "0.11425" yaw = "${pi*5.0/4.0}"/> -->
-    <!-- <xacro:dummy_rotor_arm id = "${child4}" x = "0.12427" y="-0.12427" z = "0.11425" yaw = "${pi*7.0/4.0}"/> -->
-    <xacro:dummy_rotor_arm id = "${child1}" x = "0.13427" y="0.13427" z = "0.11425" yaw = "${pi/4.0}"/>
-    <xacro:dummy_rotor_arm id = "${child2}" x = "-0.13427" y="0.13427" z = "0.11425" yaw = "${pi*3.0/4.0}"/>
-    <xacro:dummy_rotor_arm id = "${child3}" x = "-0.13427" y="-0.13427" z = "0.11425" yaw = "${pi*5.0/4.0}"/>
-    <xacro:dummy_rotor_arm id = "${child4}" x = "0.13427" y="-0.13427" z = "0.11425" yaw = "${pi*7.0/4.0}"/>
-    ## dummy link for the contact point coordinate
-    <!-- <link name="contact_point"> -->
-    <!--   <inertial> -->
-    <!--     <origin xyz="0 0 0" rpy="0 0 0"/> -->
-    <!--     <mass value="0.0001"/> -->
-    <!--     <inertia -->
-    <!--           ixx="0.000001" ixy="0.0" ixz="0.0" -->
-    <!--           iyy="0.0001" iyz="0.0" -->
-    <!--           izz="0.0001"/> -->
-    <!--     </inertial> -->
-    <!--   </link> -->
-    <!--   <joint name="cp_base_joint" type="fixed"> -->
-    <!--     <parent link="base_link"/> -->
-    <!--     <child link="contact_point"/> -->
-    <!--     <origin rpy="0 0 0" xyz="0.26 0 0"/> -->
-    <!--     <axis xyz="0 0 1"/> -->
-    <!--   </joint> -->
+    <xacro:dummy_rotor_arm id = "${child1}" x = "0.12216" y = "0.12215" z = "0.0555" yaw = "${pi/4.0}"/>
+    <xacro:dummy_rotor_arm id = "${child2}" x = "-0.12216" y = "0.12215" z = "0.0555" yaw = "${pi*3.0/4.0}"/>
+    <xacro:dummy_rotor_arm id = "${child3}" x = "-0.12216" y = "-0.12215" z = "0.0555" yaw = "${pi*5.0/4.0}"/>
+    <xacro:dummy_rotor_arm id = "${child4}" x = "0.12216" y = "-0.12215" z = "0.0555" yaw = "${pi*7.0/4.0}"/>
     <xacro:friction self="base_link"/>
   </xacro:macro>
@@ -116,11 +94,11 @@
     <link name="gimbal_link${self}">
       <inertial>
-        <origin xyz="0.022864 0.0 0.018338" rpy="0 0 0"/>
-        <mass value="0.15000"/>
-        <inertia
-            ixx="0.000063" ixy="0.000003" ixz="0.000000"
-            iyy="0.000057" iyz="0.000000"
-	    izz="0.000063"/>
-      </inertial>
+        <origin xyz="0.02375 0.00001 0.0078" rpy="0 0 0"/>  #################<!-- Changed -->
+        <mass value="0.15890"/>  #################<!-- Changed -->
+        <inertia
+          ixx="0.0000742" ixy="-0.00000005" ixz="0.0000009"
+          iyy="0.0000729" iyz="-0.00000002"
+	        izz="0.0000774"/>
+      </inertial>  #################<!-- Changed -->
       <collision>
         <origin xyz="0.0 0.0 0.0" rpy="0 0 0"/>
@@ -132,5 +110,5 @@
         <origin xyz="0 0 0" rpy="0 0 0"/>
         <geometry>
-          <mesh filename="package://gimbalrotor/urdf/beetle/mesh/beetle_hand_rotor_module.dae"/>
+          <mesh filename="package://gimbalrotor/urdf/beetle/mesh/gimbal_module.STL" scale="0.001 0.001 0.001"/>  #################<!-- Changed -->
         </geometry>
       </visual>
@@ -206,24 +184,5 @@
     </transmission>
   </xacro:macro>
-  <!-- extra_module -->
-  <!-- <xacro:macro name="extra_module" params="name parent *origin *inertial visible:=0 model_url:=0"> -->
-  <!--   <joint name="${parent}2${name}" type="fixed"> -->
-  <!--     <parent link="${parent}"/> -->
-  <!--     <child link="${name}"/> -->
-  <!--     <xacro:insert_block name="origin" /> -->
-  <!--   </joint> -->
-  <!--   <link name="${name}"> -->
-  <!--     <xacro:insert_block name="inertial" /> -->
-  <!--     <xacro:if value="${visible == 1}"> -->
-  <!--       <visual> -->
-  <!-- 	  <origin rpy="0 0 0" xyz="0 0 0"/> -->
-  <!--         <geometry> -->
-  <!--           <mesh filename="${model_url}" scale="${scale} ${scale} ${scale}"/> -->
-  <!--         </geometry> -->
-  <!--       </visual> -->
-  <!--     </xacro:if> -->
-  <!--   </link> -->
-  <!-- </xacro:macro> -->
-  ## link
+  <!-- ## link
   <link name="handbase">
     <inertial>
@@ -234,5 +193,5 @@
           ixy="0.0" ixz="0.0" iyz="0.0"/>
     </inertial>
-  </link>
+  </link> -->
   <xacro:if value="$(arg use_saw)">
     <!-- saw link  -->
@@ -291,5 +250,5 @@
     </link>
   </xacro:if>
-  ## beetle hand joint
+  <!-- ## beetle hand joint
   <joint name="handbase_baselink_joint" type="fixed">
     <child link="handbase"/>
@@ -297,18 +256,18 @@
     <origin xyz="0 0 0" rpy="0 0 0"/>
     <axis xyz="1 0 0"/>
-  </joint>
+  </joint> -->
   <xacro:if value="$(arg use_saw)">
-    <joint name="handbase_saw_joint" type="fixed">
+    <joint name="saw_joint" type="fixed">
       <child link="saw"/>
-      <parent link="handbase"/>
-      <origin xyz="0.05918 0.00052 0.08000" rpy="0 0 0"/>
+      <parent link="base_link"/>
+      <origin xyz="0.05918 0.00025 0.01700" rpy="0 0 0"/>
       <axis xyz="0 0 0"/>
     </joint>
   </xacro:if>
   <xacro:if value="$(arg use_hand)">
-    <joint name="handbase_pitchpipe_joint" type="fixed">
+    <joint name="pitchpipe_joint" type="fixed">
       <child link="passive_hand_link"/>
-      <parent link="handbase"/>
-      <origin xyz="-0.05918 0.00052 0.08000" rpy="0 0 3.142"/>
+      <parent link="base_link"/>
+      <origin xyz="-0.05918 0.00025 0.01700" rpy="0 0 3.142"/>
       <axis xyz="0 0 0"/>
     </joint>

Commit message: (URDF) passive hand with pitch joint

File: robots/gimbalrotor/urdf/beetle/gimbalrotor.urdf.xacro (robot description, xacro)
@@ -2,4 +2,6 @@
 <robot
     xmlns:xacro="http://www.ros.org/wiki/xacro" name="gimbalrotor_link" >
+  <xacro:arg name="use_saw" default="true"/>
+  <xacro:arg name="use_hand" default="true"/>
   <xacro:macro name="gimbalrotor_center_link" params="child1 child2 child3 child4">
     ## dummy
@@ -23,21 +25,21 @@
     <link name="base_link">
       <inertial>
-        <origin xyz="0.000169 0.002346 0.106123" rpy="0 0 0"/>
-        <mass value="1.400000"/>
-        <inertia
-            ixx="0.024393" ixy="0.00005" ixz="0.000015"
-	    iyy="0.024541" iyz="0.000205"
-	    izz="0.043817"/>
-      </inertial>
-      <visual>
-        <origin xyz="0 0 0" rpy="0 0 0"/>
-        <geometry>
-          <mesh filename="package://gimbalrotor/urdf/beetle/mesh/beetle_hand_base_link.dae"/>
-        </geometry>
-      </visual>
-      <collision>
-        <origin xyz="0 0 0.1065" rpy="0 0 0"/>
-        <geometry>
-          <box size="0.518 0.518 0.213"/>
+        <origin xyz="0.00193 0.00159 0.06156" rpy="0 0 0"/>  #################<!-- Changed -->
+        <mass value="1.444000"/>  #################<!-- Changed -->
+        <inertia
+          ixx="0.0368599" ixy="-0.0000221" ixz="0.0002913"
+	        iyy="0.0367152" iyz="-0.00007901"
+	        izz="0.0663418"/>
+      </inertial>  #################<!-- Changed -->
+      <visual>
+        <origin xyz="0 0 0" rpy="0 0 0"/>
+        <geometry>
+          <mesh filename="package://gimbalrotor/urdf/beetle/mesh/base_module_incenter.STL" scale="0.001 0.001 0.001"/>  #################<!-- Changed -->
+        </geometry>
+      </visual>
+      <collision>
+        <origin xyz="0 0 0.0575" rpy="0 0 0"/>
+        <geometry>
+          <box size="0.518 0.518 0.241"/>
         </geometry>
       </collision>
@@ -57,5 +59,5 @@
       <child link="fc"/>
       <parent link="base_link"/>
-      <origin rpy="0 0 0" xyz="0 0 0.12947"/>
+      <origin rpy="0 0 0" xyz="0 0 0.06927"/>  #################<!-- Changed -->
       <axis xyz="0 0 1"/>
     </joint>
@@ -81,30 +83,8 @@
       </joint>
     </xacro:macro>
-    ## dummy rotor arms
-    <!-- <xacro:dummy_rotor_arm id = "${child1}" x = "0.12427" y="0.12427" z = "0.11425" yaw = "${pi/4.0}"/> -->
-    <!-- <xacro:dummy_rotor_arm id = "${child2}" x = "-0.12427" y="0.12427" z = "0.11425" yaw = "${pi*3.0/4.0}"/> -->
-    <!-- <xacro:dummy_rotor_arm id = "${child3}" x = "-0.12427" y="-0.12427" z = "0.11425" yaw = "${pi*5.0/4.0}"/> -->
-    <!-- <xacro:dummy_rotor_arm id = "${child4}" x = "0.12427" y="-0.12427" z = "0.11425" yaw = "${pi*7.0/4.0}"/> -->
-    <xacro:dummy_rotor_arm id = "${child1}" x = "0.13427" y="0.13427" z = "0.11425" yaw = "${pi/4.0}"/>
-    <xacro:dummy_rotor_arm id = "${child2}" x = "-0.13427" y="0.13427" z = "0.11425" yaw = "${pi*3.0/4.0}"/>
-    <xacro:dummy_rotor_arm id = "${child3}" x = "-0.13427" y="-0.13427" z = "0.11425" yaw = "${pi*5.0/4.0}"/>
-    <xacro:dummy_rotor_arm id = "${child4}" x = "0.13427" y="-0.13427" z = "0.11425" yaw = "${pi*7.0/4.0}"/>
-    ## dummy link for the contact point coordinate
-    <link name="contact_point">
-      <inertial>
-        <origin xyz="0 0 0" rpy="0 0 0"/>
-        <mass value="0.0001"/>
-        <inertia
-              ixx="0.000001" ixy="0.0" ixz="0.0"
-              iyy="0.0001" iyz="0.0"
-              izz="0.0001"/>
-        </inertial>
-      </link>
-      <joint name="cp_base_joint" type="fixed">
-        <parent link="base_link"/>
-        <child link="contact_point"/>
-        <origin rpy="0 0 0" xyz="0.26 0 0"/>
-        <axis xyz="0 0 1"/>
-      </joint>
+    <xacro:dummy_rotor_arm id = "${child1}" x = "0.12216" y = "0.12215" z = "0.0555" yaw = "${pi/4.0}"/>
+    <xacro:dummy_rotor_arm id = "${child2}" x = "-0.12216" y = "0.12215" z = "0.0555" yaw = "${pi*3.0/4.0}"/>
+    <xacro:dummy_rotor_arm id = "${child3}" x = "-0.12216" y = "-0.12215" z = "0.0555" yaw = "${pi*5.0/4.0}"/>
+    <xacro:dummy_rotor_arm id = "${child4}" x = "0.12216" y = "-0.12215" z = "0.0555" yaw = "${pi*7.0/4.0}"/>
     <xacro:friction self="base_link"/>
   </xacro:macro>
@@ -114,11 +94,11 @@
     <link name="gimbal_link${self}">
       <inertial>
-        <origin xyz="0.022864 0.0 0.018338" rpy="0 0 0"/>
-        <mass value="0.15000"/>
-        <inertia
-            ixx="0.000063" ixy="0.000003" ixz="0.000000"
-            iyy="0.000057" iyz="0.000000"
-	    izz="0.000063"/>
-      </inertial>
+        <origin xyz="0.02375 0.00001 0.0078" rpy="0 0 0"/>  #################<!-- Changed -->
+        <mass value="0.15890"/>  #################<!-- Changed -->
+        <inertia
+          ixx="0.0000742" ixy="-0.00000005" ixz="0.0000009"
+          iyy="0.0000729" iyz="-0.00000002"
+	        izz="0.0000774"/>
+      </inertial>  #################<!-- Changed -->
       <collision>
         <origin xyz="0.0 0.0 0.0" rpy="0 0 0"/>
@@ -130,5 +110,5 @@
         <origin xyz="0 0 0" rpy="0 0 0"/>
         <geometry>
-          <mesh filename="package://gimbalrotor/urdf/beetle/mesh/beetle_hand_rotor_module.dae"/>
+          <mesh filename="package://gimbalrotor/urdf/beetle/mesh/gimbal_module.STL" scale="0.001 0.001 0.001"/>  #################<!-- Changed -->
         </geometry>
       </visual>
@@ -204,24 +184,15 @@
     </transmission>
   </xacro:macro>
-  <!-- extra_module -->
-  <xacro:macro name="extra_module" params="name parent *origin *inertial visible:=0 model_url:=0">
-    <joint name="${parent}2${name}" type="fixed">
-      <parent link="${parent}"/>
-      <child link="${name}"/>
-      <xacro:insert_block name="origin" />
-    </joint>
-    <link name="${name}">
-      <xacro:insert_block name="inertial" />
-      <xacro:if value="${visible == 1}">
-        <visual>
-	  <origin rpy="0 0 0" xyz="0 0 0"/>
-          <geometry>
-            <mesh filename="${model_url}" scale="${scale} ${scale} ${scale}"/>
-          </geometry>
-        </visual>
-      </xacro:if>
-    </link>
-  </xacro:macro>
-  ## link
+  <transmission name="pitch_joint">
+    <type>transmission_interface/SimpleTransmission</type>
+    <joint name="pitch_joint">
+      <hardwareInterface>hardware_interface/EffortJointInterface</hardwareInterface>
+    </joint>
+    <actuator name="pitch_joint">
+      <hardwareInterface>hardware_interface/EffortJointInterface</hardwareInterface>
+      <mechanicalReduction>1</mechanicalReduction>
+    </actuator>
+  </transmission>
+  <!-- ## link
   <link name="handbase">
     <inertial>
@@ -232,75 +203,86 @@
           ixy="0.0" ixz="0.0" iyz="0.0"/>
     </inertial>
-  </link>
-  <!-- saw link  -->
-  <link name="saw">
-    <inertial>
-      <origin xyz="0.316540 0.000030 0.036560"/>
-      <mass value="0.423690"/>
+  </link> -->
+  <xacro:if value="$(arg use_saw)">
+    <!-- saw link  -->
+    <link name="saw">
+      <inertial>
+	<origin xyz="0.31654 0.00003 0.03656"/>
+	<mass value="0.423690"/>
+	<inertia
+	    ixx="0.0004659" ixy="-0.00014505" ixz="0.0002106"
+	    iyy="0.0023921" iyz="-0.00000324"
+	    izz="0.00222804"/>
+      </inertial>
+      <visual>
+	<origin xyz="0 0 0" rpy="0 0 0"/>
+	<geometry>
+    	  <mesh filename="package://gimbalrotor/urdf/beetle/mesh/fullassem_pochitab.STL" scale="0.001 0.001 0.001"/>
+	</geometry>
+      </visual>
+      <collision>
+	<origin xyz="0.236 0.024 0.039" rpy="0 0 0"/>
+	<geometry>
+	  <box size="0.471 0.134 0.153"/>
+	</geometry>
+      </collision>
+    </link>
+  </xacro:if>
+  <xacro:if value="$(arg use_hand)">
+    <!-- pitch joint fix pipe link  -->
+    <link name="pitch_joint_link">
+      <inertial>
+        <origin xyz="0.16717 0.02381 0.00005"/>
+        <mass value="0.19260"/>
+        <inertia
+        ixx="0.0001889" ixy="0.0000569" ixz="-0.0000002"
+        iyy="0.0004543" iyz="0.0000003"
+        izz="0.0006006"/>
+      </inertial>
+      <visual>
+        <origin xyz="0 0 0" rpy="0 0 0"/>
+        <geometry>
+        <mesh filename="package://gimbalrotor/urdf/beetle/mesh/urdf_full_pitchjoint.STL" scale="1 1 1"/>
+        </geometry>
+      </visual>
+      <collision>
+        <origin xyz="0.236 0.024 0" rpy="0 0 0"/>
+        <geometry>
+      <box size="0.253 0.09 0.038"/>
+        </geometry>
+      </collision>
+    </link>
+    ## passive hand link
+    <link name="passive_hand_link">
+      <inertial>
+      <!-- <origin xyz="0.16829 0.00007 0.00007"/> <!-\- 26 or 27.5 -\-> -->
+      <!-- <mass value="0.150"/> -->
+      <!-- <inertia -->
+      <!--     ixx="0.0000323" ixy="0.0000003" ixz="-0.0000014" -->
+      <!--     iyy="0.0010134" iyz="0.000000006" -->
+      <!--     izz="0.0010082"/> -->
+      <origin xyz="0.20096 0.00005 0.00005"/> <!-- <!-\- 60 or 63 -\-> -->
+      <mass value="0.210"/>
       <inertia
-  	  ixx="0.0004659" ixy="-0.0001450" ixz="0.0002106"
-    	  iyy="0.0023921" iyz="-0.0000032"
-  	  izz="0.0022280"/>
-    </inertial>
-    <visual>
-      <origin xyz="0 0 0" rpy="0 0 0"/>
-      <geometry>
-    	<mesh filename="package://gimbalrotor/urdf/beetle/mesh/fullassem_pochitab.STL" scale="0.001 0.001 0.001"/>
-      </geometry>
-    </visual>
-    <collision>
-      <origin xyz="0.236 0.024 0.039" rpy="0 0 0"/>
-      <geometry>
-	<box size="0.471 0.134 0.153"/>
-      </geometry>
-    </collision>
-  </link>
-  <!-- pitch joint fix pipe link  -->
-  <link name="pitch_joint_link">
-    <inertial>
-      <origin xyz="0.16717 0.02381 0.00005"/>
-      <mass value="0.19260"/>
-      <inertia
-  	  ixx="0.0001889" ixy="0.0000569" ixz="-0.0000002"
-  	  iyy="0.0004543" iyz="0.0000003"
-  	  izz="0.0006006"/>
-    </inertial>
-    <visual>
-      <origin xyz="0 0 0" rpy="0 0 0"/>
-      <geometry>
-    	<mesh filename="package://gimbalrotor/urdf/beetle/mesh/urdf_full_pitchjoint.STL" scale="1 1 1"/>
-      </geometry>
-    </visual>
-    <collision>
-      <origin xyz="0.236 0.024 0" rpy="0 0 0"/>
-      <geometry>
-  	<box size="0.253 0.09 0.038"/>
-      </geometry>
-    </collision>
-  </link>
-  <!-- pitch joint hand assem  -->
-  <link name="hand_assem_link">
-    <inertial>
-      <origin xyz="0.09014 0.00038 0.02488"/>
-      <mass value="0.4820000"/>
-      <inertia
-    ixx="0.0008951" ixy="-0.0000298" ixz="0.0006735"
-    iyy="0.0052070" iyz="-0.0000100"
-    izz="0.0045551"/>
-    </inertial>
-    <visual>
-      <origin xyz="0.03658 -0.02932 0.0085" rpy="0 0 0"/>
-      <geometry>
-      <mesh filename="package://gimbalrotor/urdf/beetle/mesh/urdf_full_hand_assem.STL" scale="1 1 1"/>
-      </geometry>
-    </visual>
-    <collision>
-      <origin xyz="0.03658 -0.02307 0.0085" rpy="0 0 0"/>
-      <geometry>
-    <box size="0.5 0.1 0.177"/>
-      </geometry>
-    </collision>
-  </link>
-  ## beetle hand joint
+          ixx="0.0000946" ixy="-0.00000006" ixz="-0.0000018"
+          iyy="0.0017155" iyz="0.000000007"
+          izz="0.0016576"/>
+          </inertial>
+      <visual>
+        <origin xyz="0.027 0 0" rpy="0 0 0"/>
+        <geometry>
+          <mesh filename="package://gimbalrotor/urdf/beetle/mesh/urdf_passive_hand.STL"
+                scale="0.001 0.001 0.001"/>
+        </geometry>
+      </visual>
+      <collision>
+        <origin xyz="0.236 0.024 0" rpy="0 0 0"/>
+        <geometry>
+          <box size="0.253 0.09 0.038"/>
+        </geometry>
+      </collision>
+    </link>
+  </xacro:if>
+  <!-- ## beetle hand joint
   <joint name="handbase_baselink_joint" type="fixed">
     <child link="handbase"/>
@@ -308,63 +290,29 @@
     <origin xyz="0 0 0" rpy="0 0 0"/>
     <axis xyz="1 0 0"/>
-  </joint>
-  <joint name="handbase_saw_joint" type="fixed">
-    <child link="saw"/>
-    <parent link="handbase"/>
-    <origin xyz="0.05918 0.00052 0.08000" rpy="0 0 0"/>
-    <axis xyz="0 0 0"/>
-  </joint>
-  <joint name="handbase_pitchpipe_joint" type="fixed">
-    <child link="pitch_joint_link"/>
-    <parent link="handbase"/>
-    <origin xyz="-0.05918 0.00052 0.08000" rpy="0 0 3.142"/>
-    <axis xyz="0 0 0"/>
-  </joint>
-  <joint name="pitch_joint" type="revolute">
-    <parent link="pitch_joint_link"/>
-    <child link="hand_assem_link"/>
-    <!-- location of the pitch axis -->
-    <origin xyz="0.22074 0.02932 0" rpy="0 0 0"/>  <!-- 0.02932 is pulley origin -->
-    <axis xyz="0 1 0"/>
-    <limit effort="10" velocity="0.1" lower="-1.57" upper="1.57"/>
-    <dynamics damping="0.9" friction="0.05"/>
-  </joint>
-  <joint name="wire_joint" type="revolute">
-    <parent link="base_link"/>
-    <child link="virtual_wire"/>
-    <limit effort="10" velocity="1.0" lower="-1.57" upper="1.57"/>
-    <dynamics damping="0.1" friction="0.01"/>
-    <origin rpy="0 0 0" xyz="0 0 0"/>
-    <axis xyz="0 0 1"/>
-  </joint>
-  <link name="virtual_wire">
-    <inertial>
-      <origin xyz="0 0 0" rpy="0 0 0"/>
-      <mass value="0.00001"/>
-      <inertia
-          ixx="0.00001" ixy="0.0" ixz="0.0"
-          iyy="0.00001" iyz="0.0"
-          izz="0.00001"/>
-    </inertial>
-  </link>
-  <transmission name="pitch_joint">
-    <type>transmission_interface/SimpleTransmission</type>
-    <joint name="pitch_joint">
-      <hardwareInterface>hardware_interface/EffortJointInterface</hardwareInterface>
-    </joint>
-    <actuator name="pitch_joint">
-      <hardwareInterface>hardware_interface/EffortJointInterface</hardwareInterface>
-      <mechanicalReduction>1</mechanicalReduction>
-    </actuator>
-  </transmission>
-  <transmission name="wire_joint">
-    <type>transmission_interface/SimpleTransmission</type>
-    <joint name="wire_joint">
-      <hardwareInterface>hardware_interface/EffortJointInterface</hardwareInterface>
-    </joint>
-    <actuator name="wire_joint">
-      <hardwareInterface>hardware_interface/EffortJointInterface</hardwareInterface>
-      <mechanicalReduction>1</mechanicalReduction>
-    </actuator>
-  </transmission>
+  </joint> -->
+  <xacro:if value="$(arg use_saw)">
+    <joint name="saw_joint" type="fixed">
+      <child link="saw"/>
+      <parent link="base_link"/>
+      <origin xyz="0.05918 0.00025 0.01700" rpy="0 0 0"/>
+      <axis xyz="0 0 0"/>
+    </joint>
+  </xacro:if>
+  <xacro:if value="$(arg use_hand)">
+    <joint name="pipe_joint" type="fixed">
+      <child link="pitch_joint_link"/>
+      <parent link="base_link"/>
+      <origin xyz="-0.05918 0.00025 0.01700" rpy="0 0 3.142"/>
+      <axis xyz="0 0 0"/>
+    </joint>
+    <joint name="pitch_joint" type="revolute">
+      <parent link="pitch_joint_link"/>
+      <child link="passive_hand_link"/>
+      <!-- location of the pitch axis -->
+      <origin xyz="0.2205 0 0" rpy="0 0 0"/>  <!-- 0.02932 is pulley origin -->
+      <axis xyz="0 1 0"/>
+      <limit effort="10" velocity="0.1" lower="-1.57" upper="1.57"/>
+      <dynamics damping="0.9" friction="0.05"/>
+    </joint>
+  </xacro:if>
 </robot>
