Commit message: [PitchJoint_PassivePerching] Integrate Passive-Perching Pitch-Joint Control

File: robots/gimbalrotor/urdf/beetle/gimbalrotor.urdf.xacro (robot description, xacro)
@@ -184,14 +184,4 @@
     </transmission>
   </xacro:macro>
-  <transmission name="pitch_joint">
-    <type>transmission_interface/SimpleTransmission</type>
-    <joint name="pitch_joint">
-      <hardwareInterface>hardware_interface/EffortJointInterface</hardwareInterface>
-    </joint>
-    <actuator name="pitch_joint">
-      <hardwareInterface>hardware_interface/EffortJointInterface</hardwareInterface>
-      <mechanicalReduction>1</mechanicalReduction>
-    </actuator>
-  </transmission>
   <!-- ## link
   <link name="handbase">
@@ -282,4 +272,14 @@
         </geometry>
       </collision>
+    </link>
+    <link name="perching_center">
+      <inertial>
+        <origin xyz="0 0 0" rpy="0 0 0"/>
+        <mass value="0.00001"/>
+        <inertia
+            ixx="0.000001" ixy="0.0" ixz="0.0"
+            iyy="0.000001" iyz="0.0"
+            izz="0.000001"/>
+      </inertial>
     </link>
   </xacro:if>
@@ -315,4 +315,23 @@
       <dynamics damping="0.9" friction="0.05"/>
     </joint>
+    <joint name="perching_center_joint" type="fixed">
+      <parent link="passive_hand_link"/>
+      <child link="perching_center"/>
+      <origin xyz="0.056 0.00025 0" rpy="0 0 0"/>
+    </joint>
+    <transmission name="pitch_joint_transmission">
+      <type>transmission_interface/SimpleTransmission</type>
+      <joint name="pitch_joint">
+        <hardwareInterface>
+          hardware_interface/EffortJointInterface
+        </hardwareInterface>
+      </joint>
+      <actuator name="pitch_joint_actuator">
+        <hardwareInterface>
+          hardware_interface/EffortJointInterface
+        </hardwareInterface>
+        <mechanicalReduction>1</mechanicalReduction>
+      </actuator>
+    </transmission>
   </xacro:if>
 </robot>

Commit message: (URDF) Saw with no gear, inertia setup

File: robots/gimbalrotor/urdf/beetle/gimbalrotor.urdf.xacro (robot description, xacro)
@@ -198,15 +198,21 @@
     <link name="saw">
       <inertial>
-	<origin xyz="0.31654 0.00003 0.03656"/>
-	<mass value="0.423690"/>
+  <origin xyz="0.35108 0.0305 0.04114"/> <!-- for no gear, direct motor -->
+	<!-- <origin xyz="0.31654 0.00003 0.03656"/> --> <!-- for gear bankin-->
+	<mass value="0.37"/> <!-- for no gear, direct motor -->
+  <!-- <mass value="0.423690"/> --> <!-- for gear bankin-->
 	<inertia
-	    ixx="0.0004659" ixy="-0.00014505" ixz="0.0002106"
+      ixx="0.00050337103" ixy="-0.00027014591" ixz="0.00036440456"
+      iyy="0.00246854959" iyz="-0.00016404750"
+      izz="0.00230725723"/> <!-- for no gear, direct motor -->
+	    <!-- ixx="0.0004659" ixy="-0.00014505" ixz="0.0002106"
 	    iyy="0.0023921" iyz="-0.00000324"
-	    izz="0.00222804"/>
+	    izz="0.00222804"/> --> <!-- for gear bankin-->
       </inertial>
       <visual>
 	<origin xyz="0 0 0" rpy="0 0 0"/>
 	<geometry>
-    	  <mesh filename="package://gimbalrotor/urdf/beetle/mesh/fullassem_pochitab.STL" scale="0.001 0.001 0.001"/>
+        <mesh filename="package://gimbalrotor/urdf/beetle/mesh/urdf_saw_asm_nogear.STL" scale="0.001 0.001 0.001"/> <!-- for no gear, direct motor -->
+    	  <!-- <mesh filename="package://gimbalrotor/urdf/beetle/mesh/fullassem_pochitab.STL" scale="0.001 0.001 0.001"/> --> <!-- for gear bankin-->
 	</geometry>
       </visual>

Commit message: (URDF) Perching Hand Lock

File: robots/gimbalrotor/urdf/beetle/gimbalrotor.urdf.xacro (robot description, xacro)
@@ -235,15 +235,21 @@
 	<!--     iyy="0.0010134" iyz="0.000000006" -->
 	<!--     izz="0.0010082"/> -->
-	<origin xyz="0.20096 0.00005 0.00005"/> <!-- 60 or 63 -->
-	<mass value="0.210"/>
+	<!-- <origin xyz="0.20096 0.00005 0.00005"/> 60 or 63 -->
+	<!-- <mass value="0.210"/>
 	<inertia
 	    ixx="0.0000946" ixy="-0.00000006" ixz="-0.0000018"
 	    iyy="0.0017155" iyz="0.000000007"
-	    izz="0.0016576"/>
+	    izz="0.0016576"/> -->
+  <origin xyz="0.23313 -0.01235 0.00668"/> <!-- lock -->
+	<mass value="0.34420"/>
+	<inertia
+	    ixx="0.00044844125" ixy="0.00005346941" ixz="-0.00008531477"
+	    iyy="0.00283149126" iyz="-0.00009018516"
+	    izz="0.00288680631"/>
       </inertial>
       <visual>
 	<origin xyz="0 0 0" rpy="0 0 0"/>
 	<geometry>
-    	  <mesh filename="package://gimbalrotor/urdf/beetle/mesh/passive_perching_hand_630.STL" scale="1 1 1"/>
+    	  <mesh filename="package://gimbalrotor/urdf/beetle/mesh/perching_hand_lock.STL" scale="0.001 0.001 0.001"/>
 	</geometry>
       </visual>

Commit message: (URDF) Perching Hand Lock && Perch Point UPDATED

File: robots/gimbalrotor/urdf/beetle/gimbalrotor.urdf.xacro (robot description, xacro)
@@ -241,10 +241,10 @@
 	    iyy="0.0017155" iyz="0.000000007"
 	    izz="0.0016576"/> -->
-  <origin xyz="0.23313 -0.01235 0.00668"/> <!-- lock -->
-	<mass value="0.34420"/>
+  <origin xyz="0.23238 -0.01452 0.00876"/> <!-- lock -->
+	<mass value="0.35620"/>
 	<inertia
-	    ixx="0.00044844125" ixy="0.00005346941" ixz="-0.00008531477"
-	    iyy="0.00283149126" iyz="-0.00009018516"
-	    izz="0.00288680631"/>
+	    ixx="0.00043814302" ixy="0.00002455686" ixz="-0.00004022510"
+	    iyy="0.00282533956" iyz="-0.00006617372"
+	    izz="0.00290304284"/>
       </inertial>
       <visual>

Commit message: (URDF) Hand Servo Config

File: robots/gimbalrotor/urdf/beetle/gimbalrotor.urdf.xacro (robot description, xacro)
@@ -285,3 +285,66 @@
     </joint>
   </xacro:if>
+  <!-- Configuration-only link and joint for lock servo, index 4 -->
+  <link name="lock_servo_dummy_link"/>
+  <joint name="lock_servo_joint" type="revolute">
+    <parent link="passive_hand_link"/>
+    <child link="lock_servo_dummy_link"/>
+    <origin xyz="0 0 0" rpy="0 0 0"/>
+    <axis xyz="1 0 0"/>
+    <limit
+        lower="-6.284"
+        upper="6.284"
+        effort="2.0"
+        velocity="10.0"/>
+  </joint>
+  <!-- Configuration-only link and joint for hand servo, index 5 -->
+  <link name="hand_servo_dummy_link"/>
+  <joint name="hand_servo_joint" type="revolute">
+    <parent link="passive_hand_link"/>
+    <child link="hand_servo_dummy_link"/>
+    <origin xyz="0 0 0" rpy="0 0 0"/>
+    <axis xyz="1 0 0"/>
+    <limit
+        lower="-6.284"
+        upper="6.284"
+        effort="2.0"
+        velocity="10.0"/>
+  </joint>
+  <!-- <!-\- hand lock joint  -\-> -->
+  <!-- <link name="lock_servo_profile_link"> -->
+  <!--   <inertial> -->
+  <!--     <origin xyz="0 0 0" rpy="0 0 0"/> -->
+  <!--     <mass value="0.000001"/> -->
+  <!--     <inertia -->
+  <!--         ixx="0.000000001" ixy="0" ixz="0" -->
+  <!--         iyy="0.000000001" iyz="0" -->
+  <!--         izz="0.000000001"/> -->
+  <!--   </inertial> -->
+  <!-- </link> -->
+  <!-- <joint name="lock_joint" type="revolute"> -->
+  <!--   <parent link="passive_hand_link"/> -->
+  <!--   <child link="lock_servo_profile_link"/> -->
+  <!--   <origin xyz="0 0 0" rpy="0 0 0"/> -->
+  <!--   <axis xyz="1 0 0"/> -->
+  <!--   <limit -->
+  <!--       lower="-3.063" upper="-1.760" effort="2.0" velocity="3.0"/> -->
+  <!-- </joint> -->
+  <!-- <link name="hand_servo_profile_link"> -->
+  <!--   <inertial> -->
+  <!--     <origin xyz="0 0 0" rpy="0 0 0"/> -->
+  <!--     <mass value="0.000001"/> -->
+  <!--     <inertia -->
+  <!--         ixx="0.000000001" ixy="0" ixz="0" -->
+  <!--         iyy="0.000000001" iyz="0" -->
+  <!--         izz="0.000000001"/> -->
+  <!--   </inertial> -->
+  <!-- </link> -->
+  <!-- <joint name="hand_joint" type="revolute"> -->
+  <!--   <parent link="passive_hand_link"/> -->
+  <!--   <child link="hand_servo_profile_link"/> -->
+  <!--   <origin xyz="0 0 0" rpy="0 0 0"/> -->
+  <!--   <axis xyz="1 0 0"/> -->
+  <!--   <limit -->
+  <!--       lower="1.462" upper="3.073" effort="2.0" velocity="3.0"/> -->
+  <!-- </joint> -->
 </robot>

Commit message: (URDF) Wrench Sensor

File: robots/gimbalrotor/urdf/beetle/gimbalrotor.urdf.xacro (robot description, xacro)
@@ -2,6 +2,7 @@
 <robot
     xmlns:xacro="http://www.ros.org/wiki/xacro" name="gimbalrotor_link" >
-  <xacro:arg name="use_saw" default="true"/>
+  <xacro:arg name="use_saw" default="false"/>
   <xacro:arg name="use_hand" default="true"/>
+  <xacro:arg name="wrench_sensor" default="true"/>
   <xacro:macro name="gimbalrotor_center_link" params="child1 child2 child3 child4">
     ## dummy
@@ -262,4 +263,29 @@
     </link>
   </xacro:if>
+  <xacro:if value="$(arg wrench_sensor)">
+    <!-- saw link  -->
+    <link name="wrench_sensor">
+      <inertial>
+      <origin xyz="0.17641 0.00006 0.05725"/>
+      <mass value="0.445"/>
+      <inertia
+          ixx="0.00048898750" ixy="0.00006169827" ixz="0.00012259070"
+          iyy="0.00091748375" iyz="0.00000671401"
+          izz="0.00065255699"/>
+      </inertial>
+      <visual>
+	<origin xyz="0 0 0" rpy="0 0 0"/>
+	<geometry>
+        <mesh filename="package://gimbalrotor/urdf/beetle/mesh/wrench_sensor.STL" scale="0.001 0.001 0.001"/>
+	</geometry>
+      </visual>
+      <collision>
+	<origin xyz="0.236 0.024 0.039" rpy="0 0 0"/>
+	<geometry>
+	  <box size="0.471 0.134 0.153"/>
+	</geometry>
+      </collision>
+    </link>
+  </xacro:if>
   <!-- ## beetle hand joint
   <joint name="handbase_baselink_joint" type="fixed">
@@ -282,4 +308,12 @@
       <parent link="base_link"/>
       <origin xyz="-0.05918 0.00025 0.01700" rpy="0 0 3.142"/>
+      <axis xyz="0 0 0"/>
+    </joint>
+  </xacro:if>
+  <xacro:if value="$(arg wrench_sensor)">
+    <joint name="wrench_sensor_joint" type="fixed">
+      <child link="wrench_sensor"/>
+      <parent link="base_link"/>
+      <origin xyz="0.05918 0.00025 0.01700" rpy="0 0 0"/>
       <axis xyz="0 0 0"/>
     </joint>

Commit message: [Perching] Added Multilink Navigation & Admittance Control

File: robots/gimbalrotor/urdf/beetle/gimbalrotor.urdf.xacro (robot description, xacro)
@@ -3,6 +3,7 @@
     xmlns:xacro="http://www.ros.org/wiki/xacro" name="gimbalrotor_link" >
   <xacro:arg name="use_saw" default="false"/>
-  <xacro:arg name="use_hand" default="true"/>
-  <xacro:arg name="wrench_sensor" default="true"/>
+  <xacro:arg name="use_hand" default="false"/>
+  <xacro:arg name="wrench_sensor" default="false"/>
+  <xacro:arg name="use_pitch_joint" default="true"/>
   <xacro:macro name="gimbalrotor_center_link" params="child1 child2 child3 child4">
     ## dummy
@@ -311,4 +312,56 @@
     </joint>
   </xacro:if>
+  <xacro:if value="$(arg use_pitch_joint)">
+    <joint name="pitchpipe_joint" type="fixed">
+      <child link="pitch_pipe_link"/>
+      <parent link="base_link"/>
+      <origin xyz="-0.05918 0 0.01700" rpy="0 0 3.142"/>
+      <axis xyz="0 0 0"/>
+    </joint>
+  </xacro:if>
+  <xacro:if value="$(arg use_pitch_joint)">
+    <joint name="joint_pitch" type="revolute">
+      <limit effort="10.0" lower="${-pi/2}" upper="${pi/2}" velocity="0.1"/>
+      <parent link="pitch_pipe_link"/>
+      <child link="inter_joint_junction_link"/>
+      <origin rpy="0 0 0" xyz="0.2405 0 0"/>
+      <axis xyz="0 1 0"/>
+      <dynamics damping="0.9" friction="0.05"/>
+    </joint>
+  </xacro:if>
+  <transmission name="joint_pitch_tran">
+    <type>transmission_interface/SimpleTransmission</type>
+    <joint name="joint_pitch">
+      <!-- TODO: effort is torque, maybe position is enough -->
+      <hardwareInterface>hardware_interface/EffortJointInterface</hardwareInterface>
+    </joint>
+    <actuator name="joint_servo_pitch">
+      <!-- TODO: effort is torque, maybe position is enough -->
+      <hardwareInterface>hardware_interface/EffortJointInterface</hardwareInterface>
+      <mechanicalReduction>1</mechanicalReduction>
+    </actuator>
+  </transmission>
+  <xacro:if value="$(arg use_pitch_joint)">
+    <joint name="joint_yaw" type="revolute">
+      <limit effort="10.0" lower="${-pi/2}" upper="${pi/2}" velocity="0.1"/>
+      <parent link="inter_joint_junction_link"/>
+      <child link="yaw_hand_link"/>
+      <origin rpy="0 0 0" xyz="0.0515 0 0"/>
+      <axis xyz="0 0 1"/>
+      <dynamics damping="0.9" friction="0.05"/>
+    </joint>
+  </xacro:if>
+  <transmission name="joint_yaw_tran">
+    <type>transmission_interface/SimpleTransmission</type>
+    <joint name="joint_yaw">
+      <!-- TODO: effort is torque, maybe position is enough -->
+      <hardwareInterface>hardware_interface/EffortJointInterface</hardwareInterface>
+    </joint>
+    <actuator name="joint_servo_yaw">
+      <!-- TODO: effort is torque, maybe position is enough -->
+      <hardwareInterface>hardware_interface/EffortJointInterface</hardwareInterface>
+      <mechanicalReduction>1</mechanicalReduction>
+    </actuator>
+  </transmission>
   <xacro:if value="$(arg wrench_sensor)">
     <joint name="wrench_sensor_joint" type="fixed">

Commit message: (URDF) Added Pitch Joint Config

File: robots/gimbalrotor/urdf/beetle/gimbalrotor.urdf.xacro (robot description, xacro)
@@ -264,4 +264,79 @@
     </link>
   </xacro:if>
+  <xacro:if value="$(arg use_pitch_joint)">
+    ## passive hand link
+    <link name="pitch_pipe_link">
+      <inertial>
+  <origin xyz="0.23238 -0.01452 0.00876"/>
+	<mass value="0.001"/>
+	<inertia
+	    ixx="0.001" ixy="0.001" ixz="0.001"
+	    iyy="0.001" iyz="0.001"
+	    izz="0.001"/>
+      </inertial>
+      <visual>
+	<origin xyz="0 0 0" rpy="0 0 0"/>
+	<geometry>
+      <mesh filename="package://gimbalrotor/urdf/beetle/mesh/pitchjoint_asm.STL" scale="0.001 0.001 0.001"/>
+	</geometry>
+      </visual>
+      <collision>
+	<origin xyz="0.236 0.024 0" rpy="0 0 0"/>
+	<geometry>
+	  <box size="0.253 0.09 0.038"/>
+	</geometry>
+      </collision>
+    </link>
+  </xacro:if>
+  <xacro:if value="$(arg use_pitch_joint)">
+    ## passive hand link
+    <link name="inter_joint_junction_link">
+      <inertial>
+  <origin xyz="0.23238 -0.01452 0.00876"/>
+	<mass value="0.001"/>
+	<inertia
+      ixx="0.001" ixy="0.001" ixz="0.001"
+	    iyy="0.001" iyz="0.001"
+	    izz="0.001"/>
+      </inertial>
+      <visual>
+	<origin xyz="0.02450 0 0" rpy="0 0 0"/>
+	<geometry>
+      <mesh filename="package://gimbalrotor/urdf/beetle/mesh/inter_joint_junction_full.STL" scale="0.001 0.001 0.001"/>
+	</geometry>
+      </visual>
+      <collision>
+	<origin xyz="0.236 0.024 0" rpy="0 0 0"/>
+	<geometry>
+	  <box size="0.253 0.09 0.138"/>
+	</geometry>
+      </collision>
+    </link>
+  </xacro:if>
+  <xacro:if value="$(arg use_pitch_joint)">
+    ## passive hand link
+    <link name="yaw_hand_link">
+      <inertial>
+  <origin xyz="0.23238 -0.01452 0.00876"/>
+	<mass value="0.001"/>
+	<inertia
+	    ixx="0.001" ixy="0.001" ixz="0.001"
+	    iyy="0.001" iyz="0.001"
+	    izz="0.001"/>
+      </inertial>
+      <visual>
+	<origin xyz="0.012 0 0" rpy="0 0 0"/>
+	<geometry>
+      <mesh filename="package://gimbalrotor/urdf/beetle/mesh/yawjoint_hand_asm.STL" scale="0.001 0.001 0.001"/>
+	</geometry>
+      </visual>
+      <collision>
+	<origin xyz="0.236 0.024 0" rpy="0 0 0"/>
+	<geometry>
+	  <box size="0.253 0.09 0.038"/>
+	</geometry>
+      </collision>
+    </link>
+  </xacro:if>
   <xacro:if value="$(arg wrench_sensor)">
     <!-- saw link  -->
@@ -373,5 +448,5 @@
   </xacro:if>
   <!-- Configuration-only link and joint for lock servo, index 4 -->
-  <link name="lock_servo_dummy_link"/>
+  <!-- <link name="lock_servo_dummy_link"/>
   <joint name="lock_servo_joint" type="revolute">
     <parent link="passive_hand_link"/>
@@ -384,7 +459,7 @@
         effort="2.0"
         velocity="10.0"/>
-  </joint>
+  </joint> -->
   <!-- Configuration-only link and joint for hand servo, index 5 -->
-  <link name="hand_servo_dummy_link"/>
+  <!-- <link name="hand_servo_dummy_link"/>
   <joint name="hand_servo_joint" type="revolute">
     <parent link="passive_hand_link"/>
@@ -397,41 +472,4 @@
         effort="2.0"
         velocity="10.0"/>
-  </joint>
-  <!-- <!-\- hand lock joint  -\-> -->
-  <!-- <link name="lock_servo_profile_link"> -->
-  <!--   <inertial> -->
-  <!--     <origin xyz="0 0 0" rpy="0 0 0"/> -->
-  <!--     <mass value="0.000001"/> -->
-  <!--     <inertia -->
-  <!--         ixx="0.000000001" ixy="0" ixz="0" -->
-  <!--         iyy="0.000000001" iyz="0" -->
-  <!--         izz="0.000000001"/> -->
-  <!--   </inertial> -->
-  <!-- </link> -->
-  <!-- <joint name="lock_joint" type="revolute"> -->
-  <!--   <parent link="passive_hand_link"/> -->
-  <!--   <child link="lock_servo_profile_link"/> -->
-  <!--   <origin xyz="0 0 0" rpy="0 0 0"/> -->
-  <!--   <axis xyz="1 0 0"/> -->
-  <!--   <limit -->
-  <!--       lower="-3.063" upper="-1.760" effort="2.0" velocity="3.0"/> -->
-  <!-- </joint> -->
-  <!-- <link name="hand_servo_profile_link"> -->
-  <!--   <inertial> -->
-  <!--     <origin xyz="0 0 0" rpy="0 0 0"/> -->
-  <!--     <mass value="0.000001"/> -->
-  <!--     <inertia -->
-  <!--         ixx="0.000000001" ixy="0" ixz="0" -->
-  <!--         iyy="0.000000001" iyz="0" -->
-  <!--         izz="0.000000001"/> -->
-  <!--   </inertial> -->
-  <!-- </link> -->
-  <!-- <joint name="hand_joint" type="revolute"> -->
-  <!--   <parent link="passive_hand_link"/> -->
-  <!--   <child link="hand_servo_profile_link"/> -->
-  <!--   <origin xyz="0 0 0" rpy="0 0 0"/> -->
-  <!--   <axis xyz="1 0 0"/> -->
-  <!--   <limit -->
-  <!--       lower="1.462" upper="3.073" effort="2.0" velocity="3.0"/> -->
-  <!-- </joint> -->
+  </joint> -->
 </robot>
