Commit message: (URDF) Added yaw joint config & deleted old not used linkNjoint

File: robots/gimbalrotor/urdf/beetle/gimbalrotor.urdf.xacro (robot description, xacro)
@@ -3,6 +3,6 @@
     xmlns:xacro="http://www.ros.org/wiki/xacro" name="gimbalrotor_link" >
   <xacro:arg name="use_saw" default="true"/>
-  <xacro:arg name="use_hand" default="true"/>
-  <xacro:arg name="wrench_sensor" default="false"/>
+  <xacro:arg name="use_hand" default="false"/>
+  <xacro:arg name="use_yaw_joint" default="true"/>
   <xacro:macro name="gimbalrotor_center_link" params="child1 child2 child3 child4">
     ## dummy
@@ -230,16 +230,4 @@
     <link name="passive_hand_link">
       <inertial>
-	<!-- <origin xyz="0.16829 0.00007 0.00007"/> <!-\- 26 or 27.5 -\-> -->
-	<!-- <mass value="0.150"/> -->
-	<!-- <inertia -->
-	<!--     ixx="0.0000323" ixy="0.0000003" ixz="-0.0000014" -->
-	<!--     iyy="0.0010134" iyz="0.000000006" -->
-	<!--     izz="0.0010082"/> -->
-	<!-- <origin xyz="0.20096 0.00005 0.00005"/> 60 or 63 -->
-	<!-- <mass value="0.210"/>
-	<inertia
-	    ixx="0.0000946" ixy="-0.00000006" ixz="-0.0000018"
-	    iyy="0.0017155" iyz="0.000000007"
-	    izz="0.0016576"/> -->
   <origin xyz="0.23238 -0.01452 0.00876"/> <!-- lock -->
 	<mass value="0.35620"/>
@@ -263,29 +251,79 @@
     </link>
   </xacro:if>
-  <xacro:if value="$(arg wrench_sensor)">
-    <!-- saw link  -->
-    <link name="wrench_sensor">
-      <inertial>
-      <origin xyz="0.17641 0.00006 0.05725"/>
-      <mass value="0.445"/>
-      <inertia
-          ixx="0.00048898750" ixy="0.00006169827" ixz="0.00012259070"
-          iyy="0.00091748375" iyz="0.00000671401"
-          izz="0.00065255699"/>
-      </inertial>
-      <visual>
-	<origin xyz="0 0 0" rpy="0 0 0"/>
-	<geometry>
-        <mesh filename="package://gimbalrotor/urdf/beetle/mesh/wrench_sensor.STL" scale="0.001 0.001 0.001"/>
-	</geometry>
-      </visual>
-      <collision>
-	<origin xyz="0.236 0.024 0.039" rpy="0 0 0"/>
-	<geometry>
-	  <box size="0.471 0.134 0.153"/>
-	</geometry>
-      </collision>
-    </link>
-  </xacro:if>
+  <xacro:if value="$(arg use_yaw_joint)">
+      ## passive hand link
+      <link name="pitch_pipe_link">
+        <inertial>
+    <origin xyz="0.23238 -0.01452 0.00876"/>
+    <mass value="0.001"/>
+    <inertia
+        ixx="0.001" ixy="0.001" ixz="0.001"
+        iyy="0.001" iyz="0.001"
+        izz="0.001"/>
+        </inertial>
+        <visual>
+    <origin xyz="0 0 0" rpy="0 0 0"/>
+    <geometry>
+        <mesh filename="package://gimbalrotor/urdf/beetle/mesh/pitchjoint_asm.STL" scale="0.001 0.001 0.001"/>
+    </geometry>
+        </visual>
+        <collision>
+    <origin xyz="0.236 0.024 0" rpy="0 0 0"/>
+    <geometry>
+      <box size="0.253 0.09 0.038"/>
+    </geometry>
+        </collision>
+      </link>
+    </xacro:if>
+    <xacro:if value="$(arg use_yaw_joint)">
+      ## passive hand link
+      <link name="inter_joint_junction_link">
+        <inertial>
+    <origin xyz="0.23238 -0.01452 0.00876"/>
+    <mass value="0.001"/>
+    <inertia
+        ixx="0.001" ixy="0.001" ixz="0.001"
+        iyy="0.001" iyz="0.001"
+        izz="0.001"/>
+        </inertial>
+        <visual>
+    <origin xyz="0.02450 0 0" rpy="0 0 0"/>
+    <geometry>
+        <mesh filename="package://gimbalrotor/urdf/beetle/mesh/inter_joint_junction_full.STL" scale="0.001 0.001 0.001"/>
+    </geometry>
+        </visual>
+        <collision>
+    <origin xyz="0.236 0.024 0" rpy="0 0 0"/>
+    <geometry>
+      <box size="0.253 0.09 0.138"/>
+    </geometry>
+        </collision>
+      </link>
+    </xacro:if>
+    <xacro:if value="$(arg use_yaw_joint)">
+      ## passive hand link
+      <link name="yaw_hand_link">
+        <inertial>
+    <origin xyz="0.23238 -0.01452 0.00876"/>
+    <mass value="0.001"/>
+    <inertia
+        ixx="0.001" ixy="0.001" ixz="0.001"
+        iyy="0.001" iyz="0.001"
+        izz="0.001"/>
+        </inertial>
+        <visual>
+    <origin xyz="0.012 0 0" rpy="0 0 0"/>
+    <geometry>
+        <mesh filename="package://gimbalrotor/urdf/beetle/mesh/yawjoint_hand_asm.STL" scale="0.001 0.001 0.001"/>
+    </geometry>
+        </visual>
+        <collision>
+    <origin xyz="0.236 0.024 0" rpy="0 0 0"/>
+    <geometry>
+      <box size="0.253 0.09 0.038"/>
+    </geometry>
+        </collision>
+      </link>
+    </xacro:if>
   <!-- ## beetle hand joint
   <joint name="handbase_baselink_joint" type="fixed">
@@ -311,16 +349,8 @@
     </joint>
   </xacro:if>
-  <xacro:if value="$(arg wrench_sensor)">
-    <joint name="wrench_sensor_joint" type="fixed">
-      <child link="wrench_sensor"/>
-      <parent link="base_link"/>
-      <origin xyz="0.05918 0.00025 0.01700" rpy="0 0 0"/>
-      <axis xyz="0 0 0"/>
-    </joint>
-  </xacro:if>
   <!-- Configuration-only link and joint for lock servo, index 4 -->
   <link name="lock_servo_dummy_link"/>
   <joint name="lock_servo_joint" type="revolute">
-    <parent link="passive_hand_link"/>
+    <parent link="base_link"/>
     <child link="lock_servo_dummy_link"/>
     <origin xyz="0 0 0" rpy="0 0 0"/>
@@ -335,5 +365,5 @@
   <link name="hand_servo_dummy_link"/>
   <joint name="hand_servo_joint" type="revolute">
-    <parent link="passive_hand_link"/>
+    <parent link="base_link"/>
     <child link="hand_servo_dummy_link"/>
     <origin xyz="0 0 0" rpy="0 0 0"/>
@@ -345,40 +375,55 @@
         velocity="10.0"/>
   </joint>
-  <!-- <!-\- hand lock joint  -\-> -->
-  <!-- <link name="lock_servo_profile_link"> -->
-  <!--   <inertial> -->
-  <!--     <origin xyz="0 0 0" rpy="0 0 0"/> -->
-  <!--     <mass value="0.000001"/> -->
-  <!--     <inertia -->
-  <!--         ixx="0.000000001" ixy="0" ixz="0" -->
-  <!--         iyy="0.000000001" iyz="0" -->
-  <!--         izz="0.000000001"/> -->
-  <!--   </inertial> -->
-  <!-- </link> -->
-  <!-- <joint name="lock_joint" type="revolute"> -->
-  <!--   <parent link="passive_hand_link"/> -->
-  <!--   <child link="lock_servo_profile_link"/> -->
-  <!--   <origin xyz="0 0 0" rpy="0 0 0"/> -->
-  <!--   <axis xyz="1 0 0"/> -->
-  <!--   <limit -->
-  <!--       lower="-3.063" upper="-1.760" effort="2.0" velocity="3.0"/> -->
-  <!-- </joint> -->
-  <!-- <link name="hand_servo_profile_link"> -->
-  <!--   <inertial> -->
-  <!--     <origin xyz="0 0 0" rpy="0 0 0"/> -->
-  <!--     <mass value="0.000001"/> -->
-  <!--     <inertia -->
-  <!--         ixx="0.000000001" ixy="0" ixz="0" -->
-  <!--         iyy="0.000000001" iyz="0" -->
-  <!--         izz="0.000000001"/> -->
-  <!--   </inertial> -->
-  <!-- </link> -->
-  <!-- <joint name="hand_joint" type="revolute"> -->
-  <!--   <parent link="passive_hand_link"/> -->
-  <!--   <child link="hand_servo_profile_link"/> -->
-  <!--   <origin xyz="0 0 0" rpy="0 0 0"/> -->
-  <!--   <axis xyz="1 0 0"/> -->
-  <!--   <limit -->
-  <!--       lower="1.462" upper="3.073" effort="2.0" velocity="3.0"/> -->
-  <!-- </joint> -->
+  <xacro:if value="$(arg use_yaw_joint)">
+    <joint name="pitchpipe_joint" type="fixed">
+      <child link="pitch_pipe_link"/>
+      <parent link="base_link"/>
+      <origin xyz="-0.05918 0 0.01700" rpy="0 0 3.142"/>
+      <axis xyz="0 0 0"/>
+    </joint>
+  </xacro:if>
+  <xacro:if value="$(arg use_yaw_joint)">
+    <joint name="joint_pitch" type="revolute">
+      <limit effort="10.0" lower="${-pi/2}" upper="${pi/2}" velocity="0.1"/>
+      <parent link="pitch_pipe_link"/>
+      <child link="inter_joint_junction_link"/>
+      <origin rpy="0 0 0" xyz="0.2405 0 0"/>
+      <axis xyz="0 1 0"/>
+      <dynamics damping="0.9" friction="0.05"/>
+    </joint>
+  </xacro:if>
+  <transmission name="joint_pitch_tran">
+    <type>transmission_interface/SimpleTransmission</type>
+    <joint name="joint_pitch">
+      <!-- TODO: effort is torque, maybe position is enough -->
+      <hardwareInterface>hardware_interface/EffortJointInterface</hardwareInterface>
+    </joint>
+    <actuator name="joint_servo_pitch">
+      <!-- TODO: effort is torque, maybe position is enough -->
+      <hardwareInterface>hardware_interface/EffortJointInterface</hardwareInterface>
+      <mechanicalReduction>1</mechanicalReduction>
+    </actuator>
+  </transmission>
+  <xacro:if value="$(arg use_yaw_joint)">
+    <joint name="joint_yaw" type="revolute">
+      <limit effort="10.0" lower="${-pi/2}" upper="${pi/2}" velocity="0.1"/>
+      <parent link="inter_joint_junction_link"/>
+      <child link="yaw_hand_link"/>
+      <origin rpy="0 0 0" xyz="0.0515 0 0"/>
+      <axis xyz="0 0 1"/>
+      <dynamics damping="0.9" friction="0.05"/>
+    </joint>
+  </xacro:if>
+  <transmission name="joint_yaw_tran">
+    <type>transmission_interface/SimpleTransmission</type>
+    <joint name="joint_yaw">
+      <!-- TODO: effort is torque, maybe position is enough -->
+      <hardwareInterface>hardware_interface/EffortJointInterface</hardwareInterface>
+    </joint>
+    <actuator name="joint_servo_yaw">
+      <!-- TODO: effort is torque, maybe position is enough -->
+      <hardwareInterface>hardware_interface/EffortJointInterface</hardwareInterface>
+      <mechanicalReduction>1</mechanicalReduction>
+    </actuator>
+  </transmission>
 </robot>

Commit message: (URDF) Updated inertia

File: robots/gimbalrotor/urdf/beetle/gimbalrotor.urdf.xacro (robot description, xacro)
@@ -255,10 +255,10 @@
       <link name="pitch_pipe_link">
         <inertial>
-    <origin xyz="0.23238 -0.01452 0.00876"/>
+    <origin xyz="0.17942 0.02463 -0.00001"/>
     <mass value="0.001"/>
     <inertia
-        ixx="0.001" ixy="0.001" ixz="0.001"
-        iyy="0.001" iyz="0.001"
-        izz="0.001"/>
+        ixx="0.0002180" ixy="0.0001083" ixz="-0.0000018"
+        iyy="0.0008801" iyz="0.0000001"
+        izz="0.0010463"/>
         </inertial>
         <visual>
@@ -280,10 +280,10 @@
       <link name="inter_joint_junction_link">
         <inertial>
-    <origin xyz="0.23238 -0.01452 0.00876"/>
+    <origin xyz="-0.000392 0.005947 0.004039"/>
     <mass value="0.001"/>
     <inertia
-        ixx="0.001" ixy="0.001" ixz="0.001"
-        iyy="0.001" iyz="0.001"
-        izz="0.001"/>
+        ixx="0.000072" ixy="-0.000013" ixz="0.00001"
+        iyy="0.000077" iyz="0.000002"
+        izz="0.00008"/>
         </inertial>
         <visual>
@@ -305,10 +305,10 @@
       <link name="yaw_hand_link">
         <inertial>
-    <origin xyz="0.23238 -0.01452 0.00876"/>
+    <origin xyz="0.09876 -0.01002 0.01533"/>
     <mass value="0.001"/>
     <inertia
-        ixx="0.001" ixy="0.001" ixz="0.001"
-        iyy="0.001" iyz="0.001"
-        izz="0.001"/>
+        ixx="0.0007220" ixy="-0.0000888" ixz="-0.0004064"
+        iyy="0.0032767" iyz="-0.0000482"
+        izz="0.0031562"/>
         </inertial>
         <visual>

Commit message: [Perch Multilink] Pitch Rezero

File: robots/gimbalrotor/urdf/beetle/gimbalrotor.urdf.xacro (robot description, xacro)
@@ -256,5 +256,5 @@
         <inertial>
     <origin xyz="0.17942 0.02463 -0.00001"/>
-    <mass value="0.001"/>
+    <mass value="0.21857"/>
     <inertia
         ixx="0.0002180" ixy="0.0001083" ixz="-0.0000018"
@@ -281,5 +281,5 @@
         <inertial>
     <origin xyz="-0.000392 0.005947 0.004039"/>
-    <mass value="0.001"/>
+    <mass value="0.09014"/>
     <inertia
         ixx="0.000072" ixy="-0.000013" ixz="0.00001"
@@ -306,5 +306,5 @@
         <inertial>
     <origin xyz="0.09876 -0.01002 0.01533"/>
-    <mass value="0.001"/>
+    <mass value="0.51749"/>
     <inertia
         ixx="0.0007220" ixy="-0.0000888" ixz="-0.0004064"

Commit message: (URDF) Added roll joint config

File: robots/gimbalrotor/urdf/beetle/gimbalrotor.urdf.xacro (robot description, xacro)
@@ -4,5 +4,6 @@
   <xacro:arg name="use_saw" default="true"/>
   <xacro:arg name="use_hand" default="false"/>
-  <xacro:arg name="use_yaw_joint" default="true"/>
+  <xacro:arg name="use_yaw_joint" default="false"/>
+  <xacro:arg name="use_roll_joint" default="true"/>
   <xacro:macro name="gimbalrotor_center_link" params="child1 child2 child3 child4">
     ## dummy
@@ -42,5 +43,5 @@
         <origin xyz="0 0 0.0575" rpy="0 0 0"/>
         <geometry>
-          <box size="0.518 0.518 0.241"/>
+          <box size="0.518 0.518 0.541"/> <!-- <box size="0.518 0.518 0.241"/> -->
         </geometry>
       </collision>
@@ -326,4 +327,79 @@
       </link>
     </xacro:if>
+  <xacro:if value="$(arg use_roll_joint)">
+      ## passive hand link
+      <link name="pitch_pipe_link">
+        <inertial>
+    <origin xyz="0.17942 0.02463 -0.00001"/>
+    <mass value="0.21857"/>
+    <inertia
+        ixx="0.0002180" ixy="0.0001083" ixz="-0.0000018"
+        iyy="0.0008801" iyz="0.0000001"
+        izz="0.0010463"/>
+        </inertial>
+        <visual>
+    <origin xyz="0 0 0" rpy="0 0 0"/>
+    <geometry>
+        <mesh filename="package://gimbalrotor/urdf/beetle/mesh/pitchjoint_asm.STL" scale="0.001 0.001 0.001"/>
+    </geometry>
+        </visual>
+        <collision>
+    <origin xyz="0.236 0.024 0" rpy="0 0 0"/>
+    <geometry>
+      <box size="0.253 0.09 0.038"/>
+    </geometry>
+        </collision>
+      </link>
+    </xacro:if>
+    <xacro:if value="$(arg use_roll_joint)">
+      ## passive hand link
+      <link name="roll_joint_asm_link">
+        <inertial>
+    <origin xyz="0.01389 0.00134 -0.03377"/>
+    <mass value="0.27126"/>
+    <inertia
+        ixx="0.0002973" ixy="-0.0000149" ixz="-0.0000158"
+        iyy="0.0004041" iyz="0.0000123"
+        izz="0.0002392"/>
+        </inertial>
+        <visual>
+    <origin xyz="0.0270 0 0" rpy="0 0 0"/>
+    <geometry>
+        <mesh filename="package://gimbalrotor/urdf/beetle/mesh/roll_joint_asm.STL" scale="0.001 0.001 0.001"/>
+    </geometry>
+        </visual>
+        <collision>
+    <origin xyz="0.236 0.024 0" rpy="0 0 0"/>
+    <geometry>
+      <box size="0.253 0.09 0.138"/>
+    </geometry>
+        </collision>
+      </link>
+    </xacro:if>
+    <xacro:if value="$(arg use_roll_joint)">
+      ## passive hand link
+      <link name="roll_hand_link">
+        <inertial>
+    <origin xyz="0.17702 -0.02352 0.00828"/>
+    <mass value="0.30806"/>
+    <inertia
+        ixx="0.0004461" ixy="0.0001357" ixz="-0.0001474"
+        iyy="0.0013111" iyz="-0.0000856"
+        izz="0.0013577"/>
+        </inertial>
+        <visual>
+    <origin xyz="0 0 0" rpy="0 0 0"/>
+    <geometry>
+        <mesh filename="package://gimbalrotor/urdf/beetle/mesh/perching_hand_roll_asm.STL" scale="0.001 0.001 0.001"/>
+    </geometry>
+        </visual>
+        <collision>
+    <origin xyz="0 0 0" rpy="0 0 0"/>
+    <geometry>
+      <box size="0.253 0.09 0.038"/>
+    </geometry>
+        </collision>
+      </link>
+    </xacro:if>
   <!-- ## beetle hand joint
   <joint name="handbase_baselink_joint" type="fixed">
@@ -375,5 +451,5 @@
         velocity="10.0"/>
   </joint>
-  <xacro:if value="$(arg use_yaw_joint)">
+  <!-- <xacro:if value="$(arg use_yaw_joint)">
     <joint name="pitchpipe_joint" type="fixed">
       <child link="pitch_pipe_link"/>
@@ -396,9 +472,7 @@
     <type>transmission_interface/SimpleTransmission</type>
     <joint name="joint_pitch">
-      <!-- TODO: effort is torque, maybe position is enough -->
       <hardwareInterface>hardware_interface/EffortJointInterface</hardwareInterface>
     </joint>
     <actuator name="joint_servo_pitch">
-      <!-- TODO: effort is torque, maybe position is enough -->
       <hardwareInterface>hardware_interface/EffortJointInterface</hardwareInterface>
       <mechanicalReduction>1</mechanicalReduction>
@@ -418,9 +492,55 @@
     <type>transmission_interface/SimpleTransmission</type>
     <joint name="joint_yaw">
-      <!-- TODO: effort is torque, maybe position is enough -->
       <hardwareInterface>hardware_interface/EffortJointInterface</hardwareInterface>
     </joint>
     <actuator name="joint_servo_yaw">
-      <!-- TODO: effort is torque, maybe position is enough -->
+      <hardwareInterface>hardware_interface/EffortJointInterface</hardwareInterface>
+      <mechanicalReduction>1</mechanicalReduction>
+    </actuator>
+  </transmission> -->
+  <xacro:if value="$(arg use_roll_joint)">
+    <joint name="pitchpipe_joint" type="fixed">
+      <child link="pitch_pipe_link"/>
+      <parent link="base_link"/>
+      <origin xyz="-0.05918 0 0.01700" rpy="0 0 3.142"/>
+      <axis xyz="0 0 0"/>
+    </joint>
+  </xacro:if>
+  <xacro:if value="$(arg use_roll_joint)">
+    <joint name="joint_pitch" type="revolute">
+      <limit effort="10.0" lower="${-pi/2}" upper="${pi/2}" velocity="0.1"/>
+      <parent link="pitch_pipe_link"/>
+      <child link="roll_joint_asm_link"/>
+      <origin rpy="0 0 0" xyz="0.2405 0 0"/>
+      <axis xyz="0 1 0"/>
+      <dynamics damping="0.9" friction="0.05"/>
+    </joint>
+  </xacro:if>
+  <transmission name="joint_pitch_tran">
+    <type>transmission_interface/SimpleTransmission</type>
+    <joint name="joint_pitch">
+      <hardwareInterface>hardware_interface/EffortJointInterface</hardwareInterface>
+    </joint>
+    <actuator name="joint_servo_pitch">
+      <hardwareInterface>hardware_interface/EffortJointInterface</hardwareInterface>
+      <mechanicalReduction>1</mechanicalReduction>
+    </actuator>
+  </transmission>
+  <xacro:if value="$(arg use_roll_joint)">
+    <joint name="joint_roll" type="revolute">
+      <limit effort="10.0" lower="${-pi/2}" upper="${pi/2}" velocity="0.1"/>
+      <parent link="roll_joint_asm_link"/>
+      <child link="roll_hand_link"/>
+      <origin rpy="0 0 0" xyz="-0.001 0 -0.068"/>
+      <axis xyz="1 0 0"/>
+      <dynamics damping="0.9" friction="0.05"/>
+    </joint>
+  </xacro:if>
+  <transmission name="joint_roll_tran">
+    <type>transmission_interface/SimpleTransmission</type>
+    <joint name="joint_roll">
+      <hardwareInterface>hardware_interface/EffortJointInterface</hardwareInterface>
+    </joint>
+    <actuator name="joint_servo_roll">
       <hardwareInterface>hardware_interface/EffortJointInterface</hardwareInterface>
       <mechanicalReduction>1</mechanicalReduction>

Commit message: (URDF) for gazebo config

File: robots/gimbalrotor/urdf/beetle/gimbalrotor.urdf.xacro (robot description, xacro)
@@ -345,7 +345,7 @@
         </visual>
         <collision>
-    <origin xyz="0.236 0.024 0" rpy="0 0 0"/>
-    <geometry>
-      <box size="0.253 0.09 0.038"/>
+    <origin xyz="0.132000 0.023037 0.000000" rpy="0 0 0"/>
+    <geometry>
+      <box size="0.264001 0.108076 0.046968"/>
     </geometry>
         </collision>
@@ -370,7 +370,7 @@
         </visual>
         <collision>
-    <origin xyz="0.236 0.024 0" rpy="0 0 0"/>
-    <geometry>
-      <box size="0.253 0.09 0.138"/>
+    <origin xyz="0.030000 0.003525 -0.030994" rpy="0 0 0"/>
+    <geometry>
+      <box size="0.112001 0.071551 0.117989"/>
     </geometry>
         </collision>
@@ -395,7 +395,7 @@
         </visual>
         <collision>
-    <origin xyz="0 0 0" rpy="0 0 0"/>
-    <geometry>
-      <box size="0.253 0.09 0.038"/>
+    <origin xyz="0.139742 -0.000605 0.009999" rpy="0 0 0"/>
+    <geometry>
+      <box size="0.279486 0.140791 0.111999"/>
     </geometry>
         </collision>
@@ -534,5 +534,5 @@
       <origin rpy="0 0 0" xyz="-0.001 0 -0.068"/>
       <axis xyz="1 0 0"/>
-      <dynamics damping="0.9" friction="0.05"/>
+      <dynamics damping="0.02" friction="0.0"/>
     </joint>
   </xacro:if>

Commit message: [Pitch-only Nav] Added source code logic

File: robots/gimbalrotor/urdf/beetle/gimbalrotor.urdf.xacro (robot description, xacro)
@@ -5,5 +5,6 @@
   <xacro:arg name="use_hand" default="false"/>
   <xacro:arg name="use_yaw_joint" default="false"/>
-  <xacro:arg name="use_roll_joint" default="true"/>
+  <xacro:arg name="use_roll_joint" default="false"/>
+  <xacro:arg name="use_pitch_joint_only" default="true"/>
   <xacro:macro name="gimbalrotor_center_link" params="child1 child2 child3 child4">
     ## dummy
@@ -398,4 +399,54 @@
     <geometry>
       <box size="0.279486 0.140791 0.111999"/>
+    </geometry>
+        </collision>
+      </link>
+    </xacro:if>
+  <xacro:if value="$(arg use_pitch_joint_only)">
+      ## passive hand link
+      <link name="pitch_pipe_link">
+        <inertial>
+    <origin xyz="0.17942 0.02463 -0.00001"/>
+    <mass value="0.21857"/>
+    <inertia
+        ixx="0.0002180" ixy="0.0001083" ixz="-0.0000018"
+        iyy="0.0008801" iyz="0.0000001"
+        izz="0.0010463"/>
+        </inertial>
+        <visual>
+    <origin xyz="0 0 0" rpy="0 0 0"/>
+    <geometry>
+        <mesh filename="package://gimbalrotor/urdf/beetle/mesh/pitchjoint_asm.STL" scale="0.001 0.001 0.001"/>
+    </geometry>
+        </visual>
+        <collision>
+    <origin xyz="0.132000 0.023037 0.000000" rpy="0 0 0"/>
+    <geometry>
+      <box size="0.264001 0.108076 0.046968"/>
+    </geometry>
+        </collision>
+      </link>
+    </xacro:if>
+    <xacro:if value="$(arg use_pitch_joint_only)">
+      ## passive hand link
+      <link name="pitch_joint_only_hand_link">
+        <inertial>
+    <origin xyz="0.01389 0.00134 -0.03377"/>
+    <mass value="0.27126"/>
+    <inertia
+        ixx="0.0002973" ixy="-0.0000149" ixz="-0.0000158"
+        iyy="0.0004041" iyz="0.0000123"
+        izz="0.0002392"/>
+        </inertial>
+        <visual>
+    <origin xyz="0.0270 0 0" rpy="0 0 0"/>
+    <geometry>
+        <mesh filename="package://gimbalrotor/urdf/beetle/mesh/perching_hand_pitch_asm.STL" scale="0.001 0.001 0.001"/>
+    </geometry>
+        </visual>
+        <collision>
+    <origin xyz="0.030000 0.003525 -0.030994" rpy="0 0 0"/>
+    <geometry>
+      <box size="0.112001 0.071551 0.117989"/>
     </geometry>
         </collision>
@@ -499,5 +550,5 @@
     </actuator>
   </transmission> -->
-  <xacro:if value="$(arg use_roll_joint)">
+  <!-- <xacro:if value="$(arg use_roll_joint)">
     <joint name="pitchpipe_joint" type="fixed">
       <child link="pitch_pipe_link"/>
@@ -546,4 +597,32 @@
       <mechanicalReduction>1</mechanicalReduction>
     </actuator>
+  </transmission> -->
+  <xacro:if value="$(arg use_pitch_joint_only)">
+    <joint name="pitchpipe_joint" type="fixed">
+      <child link="pitch_pipe_link"/>
+      <parent link="base_link"/>
+      <origin xyz="-0.05918 0 0.01700" rpy="0 0 3.142"/>
+      <axis xyz="0 0 0"/>
+    </joint>
+  </xacro:if>
+  <xacro:if value="$(arg use_pitch_joint_only)">
+    <joint name="joint_pitch_only" type="revolute">
+      <limit effort="10.0" lower="${-pi/2}" upper="${pi/2}" velocity="0.1"/>
+      <parent link="pitch_pipe_link"/>
+      <child link="pitch_joint_only_hand_link"/>
+      <origin rpy="0 0 0" xyz="0.2405 0 0"/>
+      <axis xyz="0 1 0"/>
+      <dynamics damping="0.9" friction="0.05"/>
+    </joint>
+  </xacro:if>
+  <transmission name="joint_pitch_tran">
+    <type>transmission_interface/SimpleTransmission</type>
+    <joint name="joint_pitch_only">
+      <hardwareInterface>hardware_interface/EffortJointInterface</hardwareInterface>
+    </joint>
+    <actuator name="joint_servo_pitch">
+      <hardwareInterface>hardware_interface/EffortJointInterface</hardwareInterface>
+      <mechanicalReduction>1</mechanicalReduction>
+    </actuator>
   </transmission>
 </robot>
